File: hardware/kicad/AUXILIARY_POWER.kicad_sch (KiCad schematic)
At the start: 30 parts, among them U5 LM5164DDAR, U6 LM5164DDAR

Commit message: hardware: refine Rev A protection and passive selections
Parts:
- removed C18, C24: 2.2nF /50V X7R mandatory, Capacitor_SMD:C_0805_2012Metric, symbol RevA:C
- removed C19, C25: 2.2uF /100V X7R, Capacitor_SMD:C_1210_3225Metric, symbol RevA:C
- removed C20, C21, C26, C27: 22uF /25V X7R, Capacitor_SMD:C_1210_3225Metric, symbol RevA:C
- removed C22: 1nF C0G, Capacitor_SMD:C_0805_2012Metric, symbol RevA:C
- removed C23: 100pF C0G, Capacitor_SMD:C_0805_2012Metric, symbol RevA:C
- removed R69: 100k, Resistor_SMD:R_0805_2012Metric, symbol RevA:R
- removed R70: 27.4k, Resistor_SMD:R_0805_2012Metric, symbol RevA:R
- removed R71: 1M, Resistor_SMD:R_0805_2012Metric, symbol RevA:R
- removed R72: 82.5k, Resistor_SMD:R_0805_2012Metric, symbol RevA:R
- removed R73: 10k, Resistor_SMD:R_0805_2012Metric, symbol RevA:R
- removed R74: 475k, Resistor_SMD:R_0805_2012Metric, symbol RevA:R
- removed U5, U6: LM5164DDAR, Package_SO:TI_SO-PowerPAD-8, symbol RevA:LM5164DDAR
- added C30, C31, C36, C37: 22uF /25V X7R, Capacitor_SMD:C_1210_3225Metric, symbol RevA:C
- added C32, C38: 1nF C0G, Capacitor_SMD:C_0805_2012Metric, symbol RevA:C
- added C33, C39: 100pF C0G, Capacitor_SMD:C_0805_2012Metric, symbol RevA:C
- added C34: 2.2nF /50V X7R mandatory, Capacitor_SMD:C_0805_2012Metric, symbol RevA:C
- added C35: 2.2uF /100V X7R, Capacitor_SMD:C_1210_3225Metric, symbol RevA:C
- added R55: 909k, Resistor_SMD:R_0805_2012Metric, symbol RevA:R
- added R56, R57: 100k, Resistor_SMD:R_0805_2012Metric, symbol RevA:R
- added R58: 1M, Resistor_SMD:R_0805_2012Metric, symbol RevA:R
- added R59: 82.5k, Resistor_SMD:R_0805_2012Metric, symbol RevA:R
- added R60: 10k, Resistor_SMD:R_0805_2012Metric, symbol RevA:R
- added U10, U9: LM5164DDAR, Package_SO:TI_SO-PowerPAD-8, symbol RevA:LM5164DDAR
- C28: value 1nF C0G -> 2.2nF /50V X7R mandatory; MPN (none) -> C0805C222K5RACTU
- C29: value 100pF C0G -> 2.2uF /100V X7R; footprint Capacitor_SMD:C_0805_2012Metric -> Capacitor_SMD:C_1210_3225Metric; MPN (none) -> GRM32ER72A225KA35L
- L2: value 68uH / MSS1246T-683MLB candidate -> 68uH / MSS1246T-683MLB; MPN (none) -> MSS1246T-683MLB
- L3: value 47uH / MSS1246T-473MLB candidate -> 47uH / MSS1246T-473MLB; MPN (none) -> MSS1246T-473MLB
- R61: value 900k -> 1M; MPN (none) -> CRCW08051M00FKEA
- R62: value 100k -> 174k; MPN (none) -> CRCW0805174KFKEA
- R63: MPN (none) -> CRCW0805100KFKEA
- R64: value 1M -> 27.4k; MPN (none) -> CRCW080527K4FKEA
- R65: value 82.5k -> 1M; MPN (none) -> CRCW08051M00FKEA
- R66: value 10k -> 82.5k; MPN (none) -> CRCW080582K5FKEA
- R67: value 1M -> 10k; MPN (none) -> CRCW080510K0FKEA
- R68: value 175k -> 475k; MPN (none) -> CRCW0805475KFKEA
Connections:
- net AUX_EN_DRV: now also R58.2 (B), R59.1 (A), U9.3 (EN); no longer R64.2 (B), R65.1 (A)
- net AUX_EN_MCU: now also R65.2 (B), R66.1 (A), U10.3 (EN)
- net AUX_FB_DRV: now also C33.2 (B), R55.2 (B), R56.1 (A), U9.5 (FB); no longer R61.2 (B), R62.1 (A)
- net AUX_FB_MCU: now also R62.2 (B), R63.1 (A), C39.2 (B), U10.5 (FB); no longer C29.2 (B), R68.2 (B)
- net AUX_RIPPLE_DRV: now also R61.2 (B), C32.1 (A), C33.1 (A); no longer R67.2 (B)
- net AUX_RIPPLE_MCU: now also R68.2 (B), C38.1 (A), C39.1 (A); no longer C28.1 (A), C29.1 (A)
- net AUX_SW_DRV: now also C28.2 (B), R61.1 (A), U9.8 (SW); no longer R67.1 (A)
- net AUX_SW_MCU: now also R68.1 (A), C34.2 (B), U10.8 (SW)
- net BST_DRV: now also C28.1 (A), U9.7 (BST)
- net BST_MCU: now also C34.1 (A), U10.7 (BST)
- net BUS_FUSED: now also C29.1 (A), R65.1 (A), C35.1 (A), R58.1 (A), U10.2 (VIN), U9.2 (VIN); no longer R64.1 (A)
- net GND: now also C29.2 (B), R64.2 (B), R66.2 (B), C30.2 (B), C31.2 (B), C35.2 (B), C36.2 (B), C37.2 (B), R56.2 (B), R57.2 (B), R59.2 (B), U10.1 (GND), U10.9 (EP), U9.1 (GND), U9.9 (EP); no longer R62.2 (B), R65.2 (B)
- net PG_DRV: now also R60.1 (A), U9.6 (PGOOD); no longer R66.1 (A)
- net PG_MCU: now also R67.1 (A), U10.6 (PGOOD)
- net RON_DRV: now also R57.1 (A), U9.4 (RON); no longer R63.1 (A)
- net RON_MCU: now also R64.1 (A), U10.4 (RON)
- net V12_DRIVER: now also C30.1 (A), C31.1 (A), C32.2 (B), R55.1 (A); no longer R61.1 (A)
- net V3V3: now also R62.1 (A), R67.2 (B), C36.1 (A), C37.1 (A), C38.2 (B), R60.2 (B); no longer C28.2 (B), R66.2 (B), R68.1 (A)
Other:
- note added: "Feedback:1.2*(1+909k/100k)=12.108V;1.2*(1+174k/100k)=3.288V. PGOOD qualified by safety."
- note removed: "12V nominal feedback1.2*(1+900k/100k); 3.3V 1.2*(1+175k/100k). PGOOD qualified by safety."
- moved on the sheet: C28, C29, R61, R62, R63, R64, R65, R66, R67, R68
