File: hardware/kicad/CURRENT_SENSING.kicad_sch (KiCad schematic)
At the start: 25 parts, among them J11 OC diagnostic outputs / do no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, U10 INA293A1DBVR, U11 INA240A1D, U12 INA293A1DBVR, U13 INA293A1DBVR, U14 INA240A1D, U15 INA293A1DBVR, U16 INA293A1DBVR, U8 INA240A2D, U9 INA293A1DBVR

Commit message: hardware: refine Rev A protection and passive selections
Parts:
- removed C40, C42, C43, C44, C46, C47, C48: 100nF / 16V X7R, Capacitor_SMD:C_0805_2012Metric, symbol RevA:C
- removed C41, C45, C49: 1nF C0G, Capacitor_SMD:C_0805_2012Metric, symbol RevA:C
- removed J11: OC diagnostic outputs / do not load, Connector_PinHeader_2.54mm:PinHeader_1x05_P2.54mm_Vertical, symbol RevA:J5
- removed R88, R89, R90: 100R, Resistor_SMD:R_0805_2012Metric, symbol RevA:R
- removed U10, U9: INA293A1DBVR, Package_TO_SOT_SMD:SOT-23-5, symbol RevA:INA293A1DBVR
- removed U11: INA240A1D, Package_SO:SOIC-8_3.9x4.9mm_P1.27mm, symbol RevA:INA240A1D
- removed U8: INA240A2D, Package_SO:SOIC-8_3.9x4.9mm_P1.27mm, symbol RevA:INA240A2D
- added C52, C53, C54, C56, C57, C58, C60, C61: 100nF / 16V X7R, Capacitor_SMD:C_0805_2012Metric, symbol RevA:C
- added C55, C59: 1nF C0G, Capacitor_SMD:C_0805_2012Metric, symbol RevA:C
- added J8: OC diagnostic outputs / do not load, Connector_PinHeader_2.54mm:PinHeader_1x05_P2.54mm_Vertical, symbol RevA:J5
- added R82, R83, R84: 100R, Resistor_SMD:R_0805_2012Metric, symbol RevA:R
- added U17, U19, U20: INA293A1DBVR, Package_TO_SOT_SMD:SOT-23-5, symbol RevA:INA293A1DBVR
- added U18: INA240A1D, Package_SO:SOIC-8_3.9x4.9mm_P1.27mm, symbol RevA:INA240A1D
- C50: MPN (none) -> C0805C104K5RACTU
- C51: value 100nF / 16V X7R -> 1nF C0G; MPN (none) -> C0805C102J1GACTU
- U12: value INA293A1DBVR -> INA240A2D; footprint Package_TO_SOT_SMD:SOT-23-5 -> Package_SO:SOIC-8_3.9x4.9mm_P1.27mm; symbol RevA:INA293A1DBVR -> RevA:INA240A2D; MPN (none) -> INA240A2D
- U13, U16: MPN (none) -> INA293A1DBVR
- U14: value INA240A1D -> INA293A1DBVR; footprint Package_SO:SOIC-8_3.9x4.9mm_P1.27mm -> Package_TO_SOT_SMD:SOT-23-5; symbol RevA:INA240A1D -> RevA:INA293A1DBVR; MPN (none) -> INA293A1DBVR
- U15: value INA293A1DBVR -> INA240A1D; footprint Package_TO_SOT_SMD:SOT-23-5 -> Package_SO:SOIC-8_3.9x4.9mm_P1.27mm; symbol RevA:INA293A1DBVR -> RevA:INA240A1D; MPN (none) -> INA240A1D
Connections:
- net BUS_FAST_NEG: now also U14.1 (OUT), J8.2 (P2)
- net BUS_FAST_POS: now also U13.1 (OUT), J8.1 (P1)
- net BUS_I_FILTER: now also C51.1 (A), R82.2 (B)
- net BUS_I_RAW: now also U12.5 (OUT), R82.1 (A)
- net BUS_LINK: now also U12.1 (INM), U13.4 (INM), U14.3 (INP)
- net BUS_LINK_IN: now also U12.8 (INP), U13.3 (INP), U14.4 (INM)
- net CAP_FAST_NEG: now also J8.4 (P4), U17.1 (OUT); no longer U13.1 (OUT)
- net CAP_FAST_POS: now also U16.1 (OUT), J8.3 (P3); no longer U12.1 (OUT)
- net CAP_I_FILTER: now also C55.1 (A), R83.2 (B)
- net CAP_I_RAW: now also U15.5 (OUT), R83.1 (A)
- net CAP_LINK: now also U15.1 (INM), U16.4 (INM), U17.3 (INP); no longer U12.4 (INM), U13.3 (INP)
- net CAP_LINK_IN: now also U15.8 (INP), U16.3 (INP), U17.4 (INM); no longer U12.3 (INP), U13.4 (INM)
- net GND: now also U12.3 (REF2), U15.3 (REF2), C52.2 (B), C53.2 (B), C54.2 (B), C55.2 (B), C56.2 (B), C57.2 (B), C58.2 (B), C59.2 (B), C60.2 (B), C61.2 (B), J8.5 (P5), U17.2 (GND), U18.2 (GND), U18.3 (REF2), U19.2 (GND), U20.2 (GND); no longer U14.3 (REF2)
- net IL_FAST_NEG: now also U20.1 (OUT); no longer U16.1 (OUT)
- net IL_FAST_POS: now also U19.1 (OUT); no longer U15.1 (OUT)
- net IL_I_FILTER: now also C59.1 (A), R84.2 (B)
- net IL_I_RAW: now also R84.1 (A), U18.5 (OUT); no longer U14.5 (OUT)
- net IL_TO_L: now also U18.1 (INM), U19.4 (INM), U20.3 (INP); no longer U14.1 (INM), U15.4 (INM), U16.3 (INP)
- net SW_NODE_A: now also U18.8 (INP), U19.3 (INP), U20.4 (INM); no longer U14.8 (INP), U15.3 (INP), U16.4 (INM)
- net V3V3: now also U12.6 (VS), U12.7 (REF1), U14.5 (VS), U15.6 (VS), U15.7 (REF1), C52.1 (A), C53.1 (A), C54.1 (A), C56.1 (A), C57.1 (A), C58.1 (A), C60.1 (A), C61.1 (A), U17.5 (VS), U18.6 (VS), U18.7 (REF1), U19.5 (VS), U20.5 (VS); no longer C51.1 (A), U12.5 (VS), U14.6 (VS), U14.7 (REF1), U15.5 (VS)
Other:
- moved on the sheet: C50, C51, U13, U16

Commit message: hardware: define PCB harness boundary and Kelvin nets
Connections:
- net BUS_LINK renamed BUS_KELVIN_M
- net BUS_LINK_IN renamed BUS_KELVIN_P
- net CAP_LINK renamed CAP_KELVIN_M
- net CAP_LINK_IN renamed CAP_KELVIN_P
- net IL_TO_L renamed IL_KELVIN_M
- net SW_NODE_A renamed IL_KELVIN_P
Changed lines of the file:
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@@
   (generator "eeschema")
   (paper "User" 1189 841)
-  (title_block (title "CURRENT_SENSING / Prototype Rev A draft") (rev "RevA-draft") (comment 1 "ASSUMPTION - MUST VERIFY ON PROTOTYPE; no PCB placement"))
+  (title_block (title "CURRENT_SENSING / Prototype Rev A draft") (rev "RevA-draft") (comment 1 "ASSUMPTION - MUST VERIFY ON PROTOTYPE; PCB engineering authorized"))
   (symbol
     (lib_id "RevA:INA240A2D")
@@
   )
   (wire (pts (xy 73.66 110.49) (xy 68.58 110.49)) (stroke (width 0) (type default)))
-  (global_label "BUS_LINK" (shape bidirectional) (at 68.58 110.49 0) (fields_autoplaced yes) (effects (font (size 0.8 0.8))))
+  (global_label "BUS_KELVIN_M"
+    (shape bidirectional)
+    (at 68.58 110.49 0)
+    (fields_autoplaced yes)
+    (effects (font (size 0.8 0.8)))
+  )
   (wire (pts (xy 73.66 113.03) (xy 68.58 113.03)) (stroke (width 0) (type default)))
   (global_label "GND" (shape bidirectional) (at 68.58 113.03 0) (fields_autoplaced yes) (effects (font (size 0.8 0.8))))
@@
   (global_label "V3V3" (shape bidirectional) (at 109.22 115.57 180) (fields_autoplaced yes) (effects (font (size 0.8 0.8))))
   (wire (pts (xy 104.14 118.11) (xy 109.22 118.11)) (stroke (width 0) (type default)))
-  (global_label "BUS_LINK_IN"
+  (global_label "BUS_KELVIN_P"
     (shape bidirectional)
     (at 109.22 118.11 180)
@@
   (global_label "GND" (shape bidirectional) (at 678.18 114.3 0) (fields_autoplaced yes) (effects (font (size 0.8 0.8))))
   (wire (pts (xy 683.26 116.84) (xy 678.18 116.84)) (stroke (width 0) (type default)))
-  (global_label "BUS_LINK_IN"
+  (global_label "BUS_KELVIN_P"
     (shape bidirectional)
     (at 678.18 116.84 0)
@@
   )
   (wire (pts (xy 713.74 111.76) (xy 718.82 111.76)) (stroke (width 0) (type default)))
-  (global_label "BUS_LINK"
+  (global_label "BUS_KELVIN_M"
     (shape bidirectional)
     (at 718.82 111.76 180)
@@
   (global_label "GND" (shape bidirectional) (at 982.98 114.3 0) (fields_autoplaced yes) (effects (font (size 0.8 0.8))))
   (wire (pts (xy 988.06 116.84) (xy 982.98 116.84)) (stroke (width 0) (type default)))
-  (global_label "BUS_LINK"
+  (global_label "BUS_KELVIN_M"
     (shape bidirectional)
     (at 982.98 116.84 0)
@@
   )
   (wire (pts (xy 1018.54 111.76) (xy 1023.62 111.76)) (stroke (width 0) (type default)))
-  (global_label "BUS_LINK_IN"
+  (global_label "BUS_KELVIN_P"
     (shape bidirectional)
     (at 1023.62 111.76 180)
@@
   )
   (wire (pts (xy 226.06 212.09) (xy 220.98 212.09)) (stroke (width 0) (type default)))
-  (global_label "CAP_LINK"
+  (global_label "CAP_KELVIN_M"
     (shape bidirectional)
     (at 220.98 212.09 0)
@@
   (global_label "V3V3" (shape bidirectional) (at 261.62 217.17 180) (fields_autoplaced yes) (effects (font (size 0.8 0.8))))
   (wire (pts (xy 256.54 219.71) (xy 261.62 219.71)) (stroke (width 0) (type default)))
-  (global_label "CAP_LINK_IN"
+  (global_label "CAP_KELVIN_P"
     (shape bidirectional)
     (at 261.62 219.71 180)
@@
   (global_label "GND" (shape bidirectional) (at 830.58 215.9 0) (fields_autoplaced yes) (effects (font (size 0.8 0.8))))
   (wire (pts (xy 835.66 218.44) (xy 830.58 218.44)) (stroke (width 0) (type default)))
-  (global_label "CAP_LINK_IN"
+  (global_label "CAP_KELVIN_P"
     (shape bidirectional)
     (at 830.58 218.44 0)
@@
   )
   (wire (pts (xy 866.14 213.36) (xy 871.22 213.36)) (stroke (width 0) (type default)))
-  (global_label "CAP_LINK"
+  (global_label "CAP_KELVIN_M"
     (shape bidirectional)
     (at 871.22 213.36 180)
@@
   (global_label "GND" (shape bidirectional) (at 68.58 317.5 0) (fields_autoplaced yes) (effects (font (size 0.8 0.8))))
   (wire (pts (xy 73.66 320.04) (xy 68.58 320.04)) (stroke (width 0) (type default)))
-  (global_label "CAP_LINK" (shape bidirectional) (at 68.58 320.04 0) (fields_autoplaced yes) (effects (font (size 0.8 0.8))))
+  (global_label "CAP_KELVIN_M"
+    (shape bidirectional)
+    (at 68.58 320.04 0)
+    (fields_autoplaced yes)
+    (effects (font (size 0.8 0.8)))
+  )
   (wire (pts (xy 104.14 314.96) (xy 109.22 314.96)) (stroke (width 0) (type default)))
-  (global_label "CAP_LINK_IN"
+  (global_label "CAP_KELVIN_P"
     (shape bidirectional)
     (at 109.22 314.96 180)
@@
   )
   (wire (pts (xy 378.46 313.69) (xy 373.38 313.69)) (stroke (width 0) (type default)))
-  (global_label "IL_TO_L" (shape bidirectional) (at 373.38 313.69 0) (fields_autoplaced yes) (effects (font (size 0.8 0.8))))
+  (global_label "IL_KELVIN_M"
+    (shape bidirectional)
+    (at 373.38 313.69 0)
+    (fields_autoplaced yes)
+    (effects (font (size 0.8 0.8)))
+  )
   (wire (pts (xy 378.46 316.23) (xy 373.38 316.23)) (stroke (width 0) (type default)))
   (global_label "GND" (shape bidirectional) (at 373.38 316.23 0) (fields_autoplaced yes) (effects (font (size 0.8 0.8))))
@@
   (global_label "V3V3" (shape bidirectional) (at 414.02 318.77 180) (fields_autoplaced yes) (effects (font (size 0.8 0.8))))
   (wire (pts (xy 408.94 321.31) (xy 414.02 321.31)) (stroke (width 0) (type default)))
-  (global_label "SW_NODE_A"
+  (global_label "IL_KELVIN_P"
     (shape bidirectional)
     (at 414.02 321.31 180)
@@
   (global_label "GND" (shape bidirectional) (at 982.98 317.5 0) (fields_autoplaced yes) (effects (font (size 0.8 0.8))))
   (wire (pts (xy 988.06 320.04) (xy 982.98 320.04)) (stroke (width 0) (type default)))
-  (global_label "SW_NODE_A"
+  (global_label "IL_KELVIN_P"
     (shape bidirectional)
     (at 982.98 320.04 0)
@@
   )
   (wire (pts (xy 1018.54 314.96) (xy 1023.62 314.96)) (stroke (width 0) (type default)))
-  (global_label "IL_TO_L"
+  (global_label "IL_KELVIN_M"
     (shape bidirectional)
     (at 1023.62 314.96 180)
@@
   (global_label "GND" (shape bidirectional) (at 220.98 419.1 0) (fields_autoplaced yes) (effects (font (size 0.8 0.8))))
   (wire (pts (xy 226.06 421.64) (xy 220.98 421.64)) (stroke (width 0) (type default)))
-  (global_label "IL_TO_L" (shape bidirectional) (at 220.98 421.64 0) (fields_autoplaced yes) (effects (font (size 0.8 0.8))))
+  (global_label "IL_KELVIN_M"
+    (shape bidirectional)
+    (at 220.98 421.64 0)
+    (fields_autoplaced yes)
+    (effects (font (size 0.8 0.8)))
+  )
   (wire (pts (xy 256.54 416.56) (xy 261.62 416.56)) (stroke (width 0) (type default)))
-  (global_label "SW_NODE_A"
+  (global_label "IL_KELVIN_P"
     (shape bidirectional)
     (at 261.62 416.56 180)
