File: hardware/kicad/GATE_DRIVER.kicad_sch (KiCad schematic)
At the start: 30 parts, among them U1 UCC27282DRCR, U2 UCC27282DRCR, U3 SN74LVC2G08DCUR, U4 SN74LVC2G08DCUR

Commit message: hardware: refine Rev A protection and passive selections
Parts:
- removed C10, C13: 1uF /25V X7R, Capacitor_SMD:C_0805_2012Metric, symbol RevA:C
- removed C11, C14, C16, C17: 100nF / 16V X7R, Capacitor_SMD:C_0805_2012Metric, symbol RevA:C
- removed C12, C9: 470nF /25V X7R bootstrap / effectiveC>=200nF targ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, Capacitor_SMD:C_0805_2012Metric, symbol RevA:C
- removed C15: 1nF EN filter, Capacitor_SMD:C_0805_2012Metric, symbol RevA:C
- removed D13, D14: 1N4148W DNI turnoff bypass, Diode_SMD:D_SOD-123, symbol RevA:D
- removed R55, R57: 2.2R DNI turnoff option, Resistor_SMD:R_0805_2012Metric, symbol RevA:R
- removed R56: 4.7R gate / tunable, Resistor_SMD:R_0603_1608Metric, symbol RevA:R
- removed R58, R59, R60: 10k, Resistor_SMD:R_0805_2012Metric, symbol RevA:R
- removed U1, U2: UCC27282DRCR, Package_SON:VSON-10-1EP_3x3mm_P0.5mm_EP1.65x2.4mm, symbol RevA:UCC27282DRCR
- removed U3, U4: SN74LVC2G08DCUR, Package_SO:VSSOP-8_2.3x2mm_P0.5mm, symbol RevA:SN74LVC2G08DCUR
- added C19, C22: 470nF /50V X7R bootstrap / effectiveC>=200nF targ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, Capacitor_SMD:C_0805_2012Metric, symbol RevA:C
- added C20, C23: 1uF /25V X7R, Capacitor_SMD:C_0805_2012Metric, symbol RevA:C
- added C21, C24, C26, C27: 100nF / 16V X7R, Capacitor_SMD:C_0805_2012Metric, symbol RevA:C
- added C25: 1nF EN filter, Capacitor_SMD:C_0805_2012Metric, symbol RevA:C
- added D10, D9: 1N4148W DNI turnoff bypass, Diode_SMD:D_SOD-123, symbol RevA:D
- added R42, R44: 4.7R gate / tunable, Resistor_SMD:R_0603_1608Metric, symbol RevA:R
- added R43, R45: 2.2R DNI turnoff option, Resistor_SMD:R_0805_2012Metric, symbol RevA:R
- added R46, R47: 10k, Resistor_SMD:R_0805_2012Metric, symbol RevA:R
- added U5, U6: UCC27282DRCR, Package_SON:VSON-10-1EP_3x3mm_P0.5mm_EP1.65x2.4mm, symbol RevA:UCC27282DRCR
- added U7, U8: SN74LVC2G08DCUR, Package_SO:VSSOP-8_2.3x2mm_P0.5mm, symbol RevA:SN74LVC2G08DCUR
- D11, D12: MPN (none) -> 1N4148W
- R48, R50: MPN (none) -> CRCW06034R70FNEA
- R49, R51: MPN (none) -> CRCW08052R20FNEA
- R52, R53: MPN (none) -> CRCW080510K0FKEA
- R54: value 4.7R gate / tunable -> 10k; footprint Resistor_SMD:R_0603_1608Metric -> Resistor_SMD:R_0805_2012Metric; MPN (none) -> CRCW080510K0FKEA
Connections:
- net GATE_AH: now also D9.2 (A), R42.2 (B); no longer D11.2 (A), R48.2 (B)
- net GATE_AL: now also D10.2 (A), R44.2 (B); no longer D12.2 (A), R50.2 (B)
- net GATE_BH: now also D11.2 (A), R48.2 (B); no longer R54.2 (B)
- net GATE_BL: now also D12.2 (A), R50.2 (B)
- net GATE_PERMIT: now also R54.1 (A), C25.1 (A), U5.6 (EN), U6.6 (EN), U7.2 (B1), U7.6 (B2), U8.2 (B1), U8.6 (B2)
- net GND: now also R54.2 (B), C20.2 (B), C21.2 (B), C23.2 (B), C24.2 (B), C25.2 (B), C26.2 (B), C27.2 (B), R46.2 (B), R47.2 (B), U5.11 (EP), U5.9 (VSS), U6.11 (EP), U6.9 (VSS), U7.4 (GND), U8.4 (GND)
- net HB_A: now also C19.1 (A), U5.3 (HB)
- net HB_B: now also C22.1 (A), U6.3 (HB)
- net HO_A: now also R42.1 (A), R43.1 (A), U5.4 (HO); no longer R48.1 (A), R49.1 (A)
- net HO_A_FAST: now also D9.1 (K), R43.2 (B); no longer D11.1 (K), R49.2 (B)
- net HO_B: now also R48.1 (A), R49.1 (A), U6.4 (HO); no longer R54.1 (A)
- net HO_B_FAST: now also D11.1 (K), R49.2 (B)
- net LO_A: now also R44.1 (A), R45.1 (A), U5.10 (LO); no longer R50.1 (A), R51.1 (A)
- net LO_A_FAST: now also D10.1 (K), R45.2 (B); no longer D12.1 (K), R51.2 (B)
- net LO_B: now also R50.1 (A), R51.1 (A), U6.10 (LO)
- net LO_B_FAST: now also D12.1 (K), R51.2 (B)
- net PWM_AH: now also U7.1 (A1)
- net PWM_AH_SAFE: now also R46.1 (A), U5.7 (HI), U7.7 (Y1); no longer R52.1 (A)
- net PWM_AL: now also U7.5 (A2)
- net PWM_AL_SAFE: now also R47.1 (A), U5.8 (LI), U7.3 (Y2); no longer R53.1 (A)
- net PWM_BH: now also U8.1 (A1)
- net PWM_BH_SAFE: now also R52.1 (A), U6.7 (HI), U8.7 (Y1)
- net PWM_BL: now also U8.5 (A2)
- net PWM_BL_SAFE: now also R53.1 (A), U6.8 (LI), U8.3 (Y2)
- net SW_NODE_A: now also C19.2 (B), U5.5 (HS)
- net SW_NODE_B: now also C22.2 (B), U6.5 (HS)
- net V12_DRIVER: now also C20.1 (A), C21.1 (A), C23.1 (A), C24.1 (A), U5.1 (VDD), U6.1 (VDD)
- net V3V3: now also C26.1 (A), C27.1 (A), U7.8 (VCC), U8.8 (VCC)
Other:
- moved on the sheet: D11, D12, R48, R49, R50, R51, R52, R53, R54
