File: hardware/kicad/PRECHARGE.kicad_sch (KiCad schematic)
At the start: 0 parts

Commit message: hardware: implement prototype Rev A electrical schematic
Parts:
- added D3, D4, D5, D6: SS110 flyback candidate / release delay MUST VERI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, Diode_SMD:D_SMA, symbol RevA:D
- added J5: PRE_BUS external actuator+feedback, symbol RevA:J4
- added J6: BYP_BUS external actuator+feedback, symbol RevA:J4
- added J7: PRE_CAP external actuator+feedback, symbol RevA:J4
- added J8: BYP_CAP external actuator+feedback, symbol RevA:J4
- added K2: PRE_BUS external NO contact / AEV14012 candidate, symbol RevA:CONTACT
- added K3: BYP_BUS external NO contact / AEV14012 candidate, symbol RevA:CONTACT
- added K4: PRE_CAP external NO contact / AEV14012 candidate, symbol RevA:CONTACT
- added K5: BYP_CAP external NO contact / AEV14012 candidate, symbol RevA:CONTACT
- added Q10, Q13, Q4, Q7: CSD18540Q5B, Package_SON:VSONP-8-1EP_5x6_P1.27mm, symbol RevA:CSD18540Q5B
- added Q11, Q14, Q5, Q8: BC857B, Package_TO_SOT_SMD:SOT-23, symbol RevA:Q_PNP
- added Q12, Q15, Q6, Q9: BC847B, Package_TO_SOT_SMD:SOT-23, symbol RevA:Q_NPN
- added R10, R11, R15, R17, R18, R19, R23, R24, R25, R26, R30, R32, R33, R34, R38, R9: 10k, Resistor_SMD:R_0805_2012Metric, symbol RevA:R
- added R12, R20, R27, R35: 4.7k, Resistor_SMD:R_0805_2012Metric, symbol RevA:R
- added R13, R21, R28, R36: 100k, Resistor_SMD:R_0805_2012Metric, symbol RevA:R
- added R14, R22, R29, R37: 47R, Resistor_SMD:R_0805_2012Metric, symbol RevA:R
- added R16, R31: 100R / AC05 5W pulse candidate, Resistor_THT:R_Axial_Power_L25.0mm_W9.0mm_P30.48mm, symbol RevA:R
Connections:
- new net ACTUATOR_12V: D3.1 (K), D4.1 (K), D5.1 (K), D6.1 (K), J5.1 (P1), J6.1 (P1), J7.1 (P1), J8.1 (P1), K2.3 (COIL_P), K3.3 (COIL_P), K4.3 (COIL_P), K5.3 (COIL_P), Q11.2 (E), Q14.2 (E), Q5.2 (E), Q8.2 (E), R10.2 (B), R18.2 (B), R25.2 (B), R33.2 (B)
- new net BUS_ISOLATED: K2.1 (COM), K3.1 (COM)
- new net BUS_LINK_IN: K3.2 (NO), R16.2 (B)
- new net BUS_PRE_R_IN: K2.2 (NO), R16.1 (A)
- new net BYP_BUS_COIL_GATE: Q7.2 (G_DS4), R17.1 (A), R22.2 (B)
- new net BYP_BUS_COIL_M: D4.2 (A), J6.2 (P2), K3.4 (COIL_M), Q7.3 (D_DS5_6_7_8)
- new net BYP_BUS_DRIVE: R20.1 (A)
- new net BYP_BUS_FB: J6.3 (P3), R23.1 (A)
- new net BYP_BUS_NPN_C: Q9.3 (C), R19.2 (B)
- new net BYP_BUS_NPN_C_BASE: Q9.1 (B), R20.2 (B), R21.1 (A)
- new net BYP_BUS_PNP_B: Q8.1 (B), R18.1 (A), R19.1 (A)
- new net BYP_BUS_PNP_C: Q8.3 (C), R22.1 (A)
- new net BYP_CAP_COIL_GATE: Q13.2 (G_DS4), R32.1 (A), R37.2 (B)
- new net BYP_CAP_COIL_M: D6.2 (A), J8.2 (P2), K5.4 (COIL_M), Q13.3 (D_DS5_6_7_8)
- new net BYP_CAP_DRIVE: R35.1 (A)
- new net BYP_CAP_FB: J8.3 (P3), R38.1 (A)
- new net BYP_CAP_NPN_C: Q15.3 (C), R34.2 (B)
- new net BYP_CAP_NPN_C_BASE: Q15.1 (B), R35.2 (B), R36.1 (A)
- new net BYP_CAP_PNP_B: Q14.1 (B), R33.1 (A), R34.1 (A)
- new net BYP_CAP_PNP_C: Q14.3 (C), R37.1 (A)
- new net CAP_ISOLATED: K4.1 (COM), K5.1 (COM)
- new net CAP_LINK_IN: K5.2 (NO), R31.2 (B)
- new net CAP_PRE_R_IN: K4.2 (NO), R31.1 (A)
- new net GND: J5.4 (P4), J6.4 (P4), J7.4 (P4), J8.4 (P4), Q10.1 (S_DS1_2_3), Q12.2 (E), Q13.1 (S_DS1_2_3), Q15.2 (E), Q4.1 (S_DS1_2_3), Q6.2 (E), Q7.1 (S_DS1_2_3), Q9.2 (E), R13.2 (B), R17.2 (B), R21.2 (B), R24.2 (B), R28.2 (B), R32.2 (B), R36.2 (B), R9.2 (B)
- new net PRE_BUS_COIL_GATE: Q4.2 (G_DS4), R14.2 (B), R9.1 (A)
- new net PRE_BUS_COIL_M: D3.2 (A), J5.2 (P2), K2.4 (COIL_M), Q4.3 (D_DS5_6_7_8)
- new net PRE_BUS_DRIVE: R12.1 (A)
- new net PRE_BUS_FB: J5.3 (P3), R15.1 (A)
- new net PRE_BUS_NPN_C: Q6.3 (C), R11.2 (B)
- new net PRE_BUS_NPN_C_BASE: Q6.1 (B), R12.2 (B), R13.1 (A)
- new net PRE_BUS_PNP_B: Q5.1 (B), R10.1 (A), R11.1 (A)
- new net PRE_BUS_PNP_C: Q5.3 (C), R14.1 (A)
- new net PRE_CAP_COIL_GATE: Q10.2 (G_DS4), R24.1 (A), R29.2 (B)
- new net PRE_CAP_COIL_M: D5.2 (A), J7.2 (P2), K4.4 (COIL_M), Q10.3 (D_DS5_6_7_8)
- new net PRE_CAP_DRIVE: R27.1 (A)
- new net PRE_CAP_FB: J7.3 (P3), R30.1 (A)
- new net PRE_CAP_NPN_C: Q12.3 (C), R26.2 (B)
- new net PRE_CAP_NPN_C_BASE: Q12.1 (B), R27.2 (B), R28.1 (A)
- new net PRE_CAP_PNP_B: Q11.1 (B), R25.1 (A), R26.1 (A)
- new net PRE_CAP_PNP_C: Q11.3 (C), R29.1 (A)
- new net V3V3: R15.2 (B), R23.2 (B), R30.2 (B), R38.2 (B)
Other:
- note added: "470uF each; 26V/100R ideal t95=0.141s, E=0.159J. 1s timeout and delta-V<1V proposal."
- note added: "Precharge feedback is required. External actuator coil current/driver rating unresolved; not an energizable assembly."
- note added: "Separate NO isolate plus NO resistor-path and NO bypass contacts; no permanent path around isolation."
- note removed: "BUS -> resistor path -> local DC link Normally OFF bypass; delta-V / current / timeout feedback Bank link equalization via SINGLE official power port"
- note removed: "See docs/task2_decisions.md and docs/interfaces.md No electrical connectivity; no validated circuit"
- title: PRECHARGE - Task 2 Proposal -> PRECHARGE / Prototype Rev A draft

Commit message: hardware: refine Rev A protection and passive selections
Parts:
- removed D5, D6: SS110 flyback candidate / release delay MUST VERI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, Diode_SMD:D_SMA, symbol RevA:D
- removed J6: BYP_BUS external actuator+feedback, symbol RevA:J4
- removed J7: PRE_CAP external actuator+feedback, symbol RevA:J4
- removed J8: BYP_CAP external actuator+feedback, symbol RevA:J4
- removed K4: PRE_CAP external NO contact / AEV14012 candidate, symbol RevA:CONTACT
- removed K5: BYP_CAP external NO contact / AEV14012 candidate, symbol RevA:CONTACT
- removed Q12, Q15: BC847B, Package_TO_SOT_SMD:SOT-23, symbol RevA:Q_NPN
- removed Q13: CSD18540Q5B, Package_SON:VSONP-8-1EP_5x6_P1.27mm, symbol RevA:CSD18540Q5B
- removed Q14: BC857B, Package_TO_SOT_SMD:SOT-23, symbol RevA:Q_PNP
- removed R33, R34, R38: 10k, Resistor_SMD:R_0805_2012Metric, symbol RevA:R
- removed R35: 4.7k, Resistor_SMD:R_0805_2012Metric, symbol RevA:R
- removed R36: 100k, Resistor_SMD:R_0805_2012Metric, symbol RevA:R
- removed R37: 47R, Resistor_SMD:R_0805_2012Metric, symbol RevA:R
- added J4: BYP_BUS actuator+reserved diagnostic / no intrins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, symbol RevA:J4
- added U3, U4: AQZ202G / external precharge SSR, symbol RevA:AQZ202G
- D3, D4: value SS110 flyback candidate / release delay MUST VERIFY -> SMBJ18CA bidirectional coil suppression / release MUST VERIFY; footprint Diode_SMD:D_SMA -> Diode_SMD:D_SMB; MPN (none) -> SMBJ18CA
- J5: value PRE_BUS external actuator+feedback -> BYP_CAP actuator+reserved diagnostic / no intrinsic auxiliary contact
- K2: value PRE_BUS external NO contact / AEV14012 candidate -> BYP_BUS external NO contact / AEV14012 bench selection; MPN (none) -> AEV14012
- K3: value BYP_BUS external NO contact / AEV14012 candidate -> BYP_CAP external NO contact / AEV14012 bench selection; MPN (none) -> AEV14012
- Q10: value CSD18540Q5B -> BC857B; footprint Package_SON:VSONP-8-1EP_5x6_P1.27mm -> Package_TO_SOT_SMD:SOT-23; symbol RevA:CSD18540Q5B -> RevA:Q_PNP; MPN (none) -> BC857B,215
- Q11, Q8: value BC857B -> BC847B; symbol RevA:Q_PNP -> RevA:Q_NPN; MPN (none) -> BC847B,215
- Q4, Q7: value CSD18540Q5B -> BC847B; footprint Package_SON:VSONP-8-1EP_5x6_P1.27mm -> Package_TO_SOT_SMD:SOT-23; symbol RevA:CSD18540Q5B -> RevA:Q_NPN; MPN (none) -> BC847B,215
- Q5: value BC857B -> CSD18540Q5B; footprint Package_TO_SOT_SMD:SOT-23 -> Package_SON:VSONP-8-1EP_5x6_P1.27mm; symbol RevA:Q_PNP -> RevA:CSD18540Q5B; MPN (none) -> CSD18540Q5B
- Q6: value BC847B -> BC857B; symbol RevA:Q_NPN -> RevA:Q_PNP; MPN (none) -> BC857B,215
- Q9: value BC847B -> CSD18540Q5B; footprint Package_TO_SOT_SMD:SOT-23 -> Package_SON:VSONP-8-1EP_5x6_P1.27mm; symbol RevA:Q_NPN -> RevA:CSD18540Q5B; MPN (none) -> CSD18540Q5B
- R10: value 10k -> 1.5k; MPN (none) -> CRCW08051K50FKEA
- R11, R15, R23, R24, R26, R32: MPN (none) -> CRCW080510K0FKEA
- R12, R20, R27: value 4.7k -> 10k; MPN (none) -> CRCW080510K0FKEA
- R13: value 100k -> 100R / HS25 100R F / external chassis mount; footprint Resistor_SMD:R_0805_2012Metric -> (none); MPN (none) -> HS25 100R F
- R14: value 47R -> 10k; MPN (none) -> CRCW080510K0FKEA
- R16: value 100R / AC05 5W pulse candidate -> 10k; footprint Resistor_THT:R_Axial_Power_L25.0mm_W9.0mm_P30.48mm -> Resistor_SMD:R_0805_2012Metric; MPN (none) -> CRCW080510K0FKEA
- R17: value 10k -> 4.7k; MPN (none) -> CRCW08054K70FKEA
- R18, R30: value 10k -> 100k; MPN (none) -> CRCW0805100KFKEA
- R19: value 10k -> 47R; MPN (none) -> CRCW080547R0FKEA
- R21: value 100k -> 150R; MPN (none) -> CRCW0805150RFKEA
- R22: value 47R -> 1.5k; MPN (none) -> CRCW08051K50FKEA
- R25: value 10k -> 100R / HS25 100R F / external chassis mount; footprint Resistor_SMD:R_0805_2012Metric -> (none); MPN (none) -> HS25 100R F
- R28: value 100k -> 10k; MPN (none) -> CRCW080510K0FKEA
- R29: value 47R -> 4.7k; MPN (none) -> CRCW08054K70FKEA
- R31: value 100R / AC05 5W pulse candidate -> 47R; footprint Resistor_THT:R_Axial_Power_L25.0mm_W9.0mm_P30.48mm -> Resistor_SMD:R_0805_2012Metric; MPN (none) -> CRCW080547R0FKEA
- R9: value 10k -> 150R; MPN (none) -> CRCW0805150RFKEA
Connections:
- net PRE_CAP_COIL_M is gone; now on net BYP_CAP_PNP_C: Q10.3 (C)
- net PRE_CAP_NPN_C is gone; now on net GND: R26.2 (B)
- net ACTUATOR_12V: now also Q10.2 (E), Q6.2 (E), R15.2 (B), R27.2 (B), J4.1 (P1); no longer Q11.2 (E), Q5.2 (E), Q8.2 (E), R10.2 (B), R18.2 (B), R25.2 (B)
- net BUS_ISOLATED: now also U3.3 (ACDC_A); no longer K3.1 (COM)
- net BUS_LINK_IN: now also K2.2 (NO), R13.2 (B); no longer K3.2 (NO), R16.2 (B)
- net BUS_PRE_R_IN: now also R13.1 (A), U3.4 (ACDC_B); no longer K2.2 (NO), R16.1 (A)
- net BYP_BUS_COIL_GATE: now also Q5.2 (G_DS4), R14.1 (A), R19.2 (B); no longer Q7.2 (G_DS4), R17.1 (A), R22.2 (B)
- net BYP_BUS_COIL_M: now also D3.2 (A), K2.4 (COIL_M), Q5.3 (D_DS5_6_7_8), J4.2 (P2); no longer D4.2 (A), K3.4 (COIL_M), Q7.3 (D_DS5_6_7_8)
- net BYP_BUS_DRIVE: now also R17.1 (A); no longer R20.1 (A)
- net BYP_BUS_FB: now also R20.1 (A), J4.3 (P3); no longer R23.1 (A)
- net BYP_BUS_NPN_C: now also Q7.3 (C), R16.2 (B); no longer Q9.3 (C), R19.2 (B)
- net BYP_BUS_NPN_C_BASE: now also Q7.1 (B), R17.2 (B), R18.1 (A); no longer Q9.1 (B), R20.2 (B), R21.1 (A)
- net BYP_BUS_PNP_B: now also Q6.1 (B), R15.1 (A), R16.1 (A); no longer Q8.1 (B), R18.1 (A), R19.1 (A)
- net BYP_BUS_PNP_C: now also Q6.3 (C), R19.1 (A); no longer Q8.3 (C), R22.1 (A)
- net BYP_CAP_COIL_GATE: now also Q9.2 (G_DS4), R26.1 (A), R31.2 (B); no longer R32.1 (A)
- net BYP_CAP_COIL_M: now also D4.2 (A), J5.2 (P2), K3.4 (COIL_M), Q9.3 (D_DS5_6_7_8)
- net BYP_CAP_DRIVE: now also R29.1 (A)
- net BYP_CAP_FB: now also J5.3 (P3), R32.1 (A)
- net BYP_CAP_NPN_C: now also Q11.3 (C), R28.2 (B)
- net BYP_CAP_NPN_C_BASE: now also Q11.1 (B), R29.2 (B), R30.1 (A)
- net BYP_CAP_PNP_B: now also Q10.1 (B), R27.1 (A), R28.1 (A)
- net BYP_CAP_PNP_C: now also R31.1 (A)
- net CAP_ISOLATED: now also K3.1 (COM), U4.3 (ACDC_A)
- net CAP_LINK_IN: now also K3.2 (NO), R25.2 (B); no longer R31.2 (B)
- net CAP_PRE_R_IN: now also R25.1 (A), U4.4 (ACDC_B); no longer R31.1 (A)
- net GND: now also Q11.2 (E), Q4.2 (E), Q5.1 (S_DS1_2_3), Q7.2 (E), Q8.2 (E), Q9.1 (S_DS1_2_3), R11.2 (B), R12.2 (B), R14.2 (B), R18.2 (B), R20.2 (B), R23.2 (B), R30.2 (B), J4.4 (P4); no longer Q10.1 (S_DS1_2_3), Q4.1 (S_DS1_2_3), Q6.2 (E), Q7.1 (S_DS1_2_3), Q9.2 (E), R13.2 (B), R17.2 (B), R21.2 (B), R28.2 (B), R9.2 (B)
- net PRE_BUS_DRIVE: now also R10.1 (A); no longer R12.1 (A)
- net PRE_BUS_FB: now also R12.1 (A); no longer J5.3 (P3), R15.1 (A)
- net PRE_CAP_DRIVE: now also R22.1 (A); no longer R27.1 (A)
- net PRE_CAP_FB: now also R24.1 (A); no longer R30.1 (A)
- net V3V3: now also R21.1 (A), R9.1 (A); no longer R15.2 (B), R23.2 (B), R30.2 (B)
- removed net PRE_BUS_COIL_GATE: Q4.2 (G_DS4), R14.2 (B), R9.1 (A)
- removed net PRE_BUS_COIL_M: D3.2 (A), J5.2 (P2), K2.4 (COIL_M), Q4.3 (D_DS5_6_7_8)
- removed net PRE_BUS_NPN_C: Q6.3 (C), R11.2 (B)
- removed net PRE_BUS_NPN_C_BASE: Q6.1 (B), R12.2 (B), R13.1 (A)
- removed net PRE_BUS_PNP_B: Q5.1 (B), R10.1 (A), R11.1 (A)
- removed net PRE_BUS_PNP_C: Q5.3 (C), R14.1 (A)
- removed net PRE_CAP_COIL_GATE: Q10.2 (G_DS4), R24.1 (A), R29.2 (B)
- removed net PRE_CAP_NPN_C_BASE: R27.2 (B), R28.1 (A)
- removed net PRE_CAP_PNP_B: Q11.1 (B), R25.1 (A), R26.1 (A)
- removed net PRE_CAP_PNP_C: Q11.3 (C), R29.1 (A)
- new net PRE_BUS_LED_M: Q4.3 (C), U3.1 (LED_M)
- new net PRE_BUS_LED_P: R9.2 (B), U3.2 (LED_P)
- new net PRE_BUS_SSR_BASE: Q4.1 (B), R10.2 (B), R11.1 (A)
- new net PRE_CAP_LED_M: Q8.3 (C), U4.1 (LED_M)
- new net PRE_CAP_LED_P: R21.2 (B), U4.2 (LED_P)
- new net PRE_CAP_SSR_BASE: Q8.1 (B), R22.2 (B), R23.1 (A)
Other:
- note added: "PRE_BUS SSR has no auxiliary contact: infer conduction using raw/link ADC; FB pin reserved LOW, not confirmation."
- note added: "PRE_CAP SSR has no auxiliary contact: infer conduction using raw/link ADC; FB pin reserved LOW, not confirmation."
- note added: "SSR path acceptance uses link voltage progression and open-path diagnosis; no resistor-only bank charge."
- note added: "Six470uF per link; 26V/100R t95 nominal0.845s, worst target<1.1s. Timeout3s and delta-V<1V."
- note removed: "470uF each; 26V/100R ideal t95=0.141s, E=0.159J. 1s timeout and delta-V<1V proposal."
- note removed: "Precharge feedback is required. External actuator coil current/driver rating unresolved; not an energizable assembly."
- moved on the sheet: D3, D4, J5, K2, K3, Q10, Q11, Q4, Q5, Q6, Q8, Q9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
