File: hardware/kicad/SAFE_DISCHARGE.kicad_sch (KiCad schematic)
At the start: 15 parts, among them J18 KEYED service meter / rated d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, Q24 CSD18540Q5B, Q25 BC857B, Q26 BC847B

Commit message: hardware: refine Rev A protection and passive selections
Parts:
- removed D26: BZT52H-C15, Diode_SMD:D_SOD-123F, symbol RevA:D
- removed D27: red residual-energy indicator / bank-powered, LED_SMD:LED_0805_2012Metric, symbol RevA:LED
- removed J18: KEYED service meter / rated discharge tool connec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, symbol RevA:J2
- removed Q24: CSD18540Q5B, Package_SON:VSONP-8-1EP_5x6_P1.27mm, symbol RevA:CSD18540Q5B
- removed Q25: BC857B, Package_TO_SOT_SMD:SOT-23, symbol RevA:Q_PNP
- removed Q26: BC847B, Package_TO_SOT_SMD:SOT-23, symbol RevA:Q_NPN
- removed R152: 10k /1W permanent bleed, Resistor_SMD:R_2512_6332Metric, symbol RevA:R
- removed R153: 100R /HS25 25W chassis mount candidate, symbol RevA:R
- removed R154, R156: 10k, Resistor_SMD:R_0805_2012Metric, symbol RevA:R
- removed R155: 47R, Resistor_SMD:R_0805_2012Metric, symbol RevA:R
- added D24: BZT52H-C15, Diode_SMD:D_SOD-123F, symbol RevA:D
- added D25: red residual-energy indicator / bank-powered, LED_SMD:LED_0805_2012Metric, symbol RevA:LED
- added J15: KEYED service meter / rated discharge tool connec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, symbol RevA:J2
- added Q20: CSD18540Q5B, Package_SON:VSONP-8-1EP_5x6_P1.27mm, symbol RevA:CSD18540Q5B
- added Q21: BC857B, Package_TO_SOT_SMD:SOT-23, symbol RevA:Q_PNP
- added Q22: BC847B, Package_TO_SOT_SMD:SOT-23, symbol RevA:Q_NPN
- added R161, R162: 10k, Resistor_SMD:R_0805_2012Metric, symbol RevA:R
- added R163: 4.7k, Resistor_SMD:R_0805_2012Metric, symbol RevA:R
- added R164: 100k, Resistor_SMD:R_0805_2012Metric, symbol RevA:R
- added R165: 22k /0.25W, Resistor_SMD:R_0805_2012Metric, symbol RevA:R
- added R166: 100R / HS25 100R F / external service tool, symbol RevA:R
- added U32: Blue Sea6006 / external independent service tool;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, symbol RevA:DISCONNECT
- R157: value 10k -> 10k /1W permanent bleed; footprint Resistor_SMD:R_0805_2012Metric -> Resistor_SMD:R_2512_6332Metric; MPN (none) -> CRCW251210K0FKEG
- R158: value 4.7k -> 100R /HS25 100R F / external chassis mount; footprint Resistor_SMD:R_0805_2012Metric -> (none); MPN (none) -> HS25 100R F
- R159: value 100k -> 10k; MPN (none) -> CRCW080510K0FKEA
- R160: value 22k /0.25W -> 47R; MPN (none) -> CRCW080547R0FKEA
Connections:
- net BANK_P_RAW: now also R157.1 (A), R158.1 (A), J15.1 (P1), R165.1 (A), U32.1 (COM); no longer R160.1 (A)
- net DUMP_DRAIN: now also R158.2 (B), Q20.3 (D_DS5_6_7_8)
- net DUMP_DRIVE: now also R163.1 (A); no longer R158.1 (A)
- net DUMP_GATE: now also R159.1 (A), R160.2 (B), D24.1 (K), Q20.2 (G_DS4)
- net DUMP_NPN_C: now also Q22.3 (C), R162.2 (B); no longer R157.2 (B)
- net DUMP_NPN_C_BASE: now also Q22.1 (B), R163.2 (B), R164.1 (A); no longer R158.2 (B), R159.1 (A)
- net DUMP_PNP_B: now also Q21.1 (B), R161.1 (A), R162.1 (A); no longer R157.1 (A)
- net DUMP_PNP_C: now also R160.1 (A), Q21.3 (C)
- net GND: now also R157.2 (B), D24.2 (A), D25.1 (K), J15.2 (P2), Q20.1 (S_DS1_2_3), Q22.2 (E), R164.2 (B), R166.2 (B)
- net RESIDUAL_LED_A: now also D25.2 (A), R165.2 (B); no longer R160.2 (B)
- net V12_DRIVER: now also Q21.2 (E), R161.2 (B)
- new net SERVICE_R_IN: R166.1 (A), U32.2 (SWITCHED)
Other:
- moved on the sheet: R157, R158, R159, R160
