File: hardware/kicad/TEMPERATURE_SENSING.kicad_sch (KiCad schematic)
At the start: 12 parts, among them J12 FET NTC probe option, J13 L NTC probe option, J14 BANK NTC probe option

Commit message: hardware: refine Rev A protection and passive selections
Parts:
- removed C59, C60, C61: 10nF, Capacitor_SMD:C_0805_2012Metric, symbol RevA:C
- removed J12: FET NTC probe option, Connector_PinHeader_2.54mm:PinHeader_1x02_P2.54mm_Vertical, symbol RevA:J2
- removed J13: L NTC probe option, Connector_PinHeader_2.54mm:PinHeader_1x02_P2.54mm_Vertical, symbol RevA:J2
- removed J14: BANK NTC probe option, Connector_PinHeader_2.54mm:PinHeader_1x02_P2.54mm_Vertical, symbol RevA:J2
- removed R116, R118, R120: 10k /1%, Resistor_SMD:R_0805_2012Metric, symbol RevA:R
- removed R117, R119, R121: NTCLE100E3103JB0 /10k NTC B3977, Connector_PinHeader_2.54mm:PinHeader_1x02_P2.54mm_Vertical, symbol RevA:R
- added C69, C70, C71: 10nF, Capacitor_SMD:C_0805_2012Metric, symbol RevA:C
- added J10: L NTC probe option, Connector_PinHeader_2.54mm:PinHeader_1x02_P2.54mm_Vertical, symbol RevA:J2
- added J11: BANK NTC probe option, Connector_PinHeader_2.54mm:PinHeader_1x02_P2.54mm_Vertical, symbol RevA:J2
- added J9: FET NTC probe option, Connector_PinHeader_2.54mm:PinHeader_1x02_P2.54mm_Vertical, symbol RevA:J2
- added R110, R112, R114: 10k /1%, Resistor_SMD:R_0805_2012Metric, symbol RevA:R
- added R111, R113, R115: NTCLE100E3103JB0 /10k NTC B3977, Connector_PinHeader_2.54mm:PinHeader_1x02_P2.54mm_Vertical, symbol RevA:R
Connections:
- net GND: now also C69.2 (B), C70.2 (B), C71.2 (B), J10.2 (P2), J11.2 (P2), J9.2 (P2), R111.2 (B), R113.2 (B), R115.2 (B)
- net TEMP_BANK_FILTER: now also C71.1 (A), J11.1 (P1), R114.2 (B), R115.1 (A)
- net TEMP_FET_FILTER: now also C69.1 (A), J9.1 (P1), R110.2 (B), R111.1 (A)
- net TEMP_L_FILTER: now also C70.1 (A), J10.1 (P1), R112.2 (B), R113.1 (A)
- net V3V3: now also R110.1 (A), R112.1 (A), R114.1 (A)
