File: hardware/kicad/VOLTAGE_SENSING.kicad_sch (KiCad schematic)
At the start: 46 parts, among them U17 TLV431AIDBZR, U18 TMUX1511PWR, U19 TMUX1511PWR, U20 TMUX1511PWR

Commit message: hardware: refine Rev A protection and passive selections
Parts:
- removed C52, C53, C54, C55: 4.7nF C0G, Capacitor_SMD:C_0805_2012Metric, symbol RevA:C
- removed C56, C57, C58: 100nF / 16V X7R, Capacitor_SMD:C_0805_2012Metric, symbol RevA:C
- removed D23, D24: 1N4148W /100V, Diode_SMD:D_SOD-123, symbol RevA:D
- removed R110, R111, R112, R113, R114, R115: 100k off leakage drain, Resistor_SMD:R_0805_2012Metric, symbol RevA:R
- removed U17: TLV431AIDBZR, Package_TO_SOT_SMD:SOT-23, symbol RevA:TLV431AIDBZR
- removed U18, U19, U20: TMUX1511PWR, Package_SO:TSSOP-14_4.4x5mm_P0.65mm, symbol RevA:TMUX1511PWR
- added C62, C63, C64, C65: 4.7nF C0G, Capacitor_SMD:C_0805_2012Metric, symbol RevA:C
- added C66, C67, C68: 100nF / 16V X7R, Capacitor_SMD:C_0805_2012Metric, symbol RevA:C
- added D13: BAT54H signal clamp, Diode_SMD:D_SOD-123F, symbol RevA:D
- added D14: BAT54H negative clamp, Diode_SMD:D_SOD-123F, symbol RevA:D
- added R85, R86, R88, R89: 33k /1%, Resistor_SMD:R_0805_2012Metric, symbol RevA:R
- added R87: 5.1k /1%, Resistor_SMD:R_0805_2012Metric, symbol RevA:R
- added R90: 6.8k /1%, Resistor_SMD:R_0805_2012Metric, symbol RevA:R
- added U21: TLV431AIDBZR, Package_TO_SOT_SMD:SOT-23, symbol RevA:TLV431AIDBZR
- added U22, U23, U24: TMUX1511PWR, Package_SO:TSSOP-14_4.4x5mm_P0.65mm, symbol RevA:TMUX1511PWR
- D15, D16, D17, D18, D19, D20: MPN (none) -> BAT54H
- D21: value BAT54H signal clamp -> 1N4148W /100V; footprint Diode_SMD:D_SOD-123F -> Diode_SMD:D_SOD-123; MPN (none) -> 1N4148W
- D22: value BAT54H negative clamp -> 1N4148W /100V; footprint Diode_SMD:D_SOD-123F -> Diode_SMD:D_SOD-123; MPN (none) -> 1N4148W
- R100, R101: value 33k /1% -> 100k off leakage drain; MPN (none) -> CRCW0805100KFKEA
- R102: value 6.8k /1% -> 100k off leakage drain; MPN (none) -> CRCW0805100KFKEA
- R103: value 3.3k /1W -> 100k off leakage drain; footprint Resistor_SMD:R_2512_6332Metric -> Resistor_SMD:R_0805_2012Metric; MPN (none) -> CRCW0805100KFKEA
- R104: value 11.8k /1% -> 100k off leakage drain; MPN (none) -> CRCW0805100KFKEA
- R105: value 10k /1% -> 100k off leakage drain; MPN (none) -> CRCW0805100KFKEA
- R106, R107, R108, R109: MPN (none) -> CRCW0805100KFKEA
- R91, R92, R94, R95: MPN (none) -> CRCW080533K0FKEA
- R93: MPN (none) -> CRCW08055K10FKEA
- R96: MPN (none) -> CRCW08056K80FKEA
- R97: value 33k /1% -> 3.3k /1W; footprint Resistor_SMD:R_0805_2012Metric -> Resistor_SMD:R_2512_6332Metric; MPN (none) -> CRCW25123K30FKEG
- R98: value 33k /1% -> 11.8k /1%; MPN (none) -> CRCW080511K8FKEA
- R99: value 5.1k /1% -> 10k /1%; MPN (none) -> CRCW080510K0FKEA
Connections:
- net ADC_CLAMP_2V7: now also R97.2 (B), R98.1 (A), D13.1 (K), U21.2 (K); no longer D21.1 (K), R103.2 (B), R104.1 (A)
- net BANK_P_RAW: now also D22.2 (A), R94.1 (A); no longer R100.1 (A)
- net BUS_DIV_TOP: now also R85.2 (B), R86.1 (A); no longer R91.2 (B), R92.1 (A)
- net BUS_FUSED: now also D21.2 (A), R91.1 (A); no longer R97.1 (A)
- net BUS_I_ADC: now also R104.1 (A), U23.3 (D1)
- net BUS_I_FILTER: now also U23.2 (S1)
- net BUS_LINK: now also R85.1 (A); no longer R91.1 (A)
- net BUS_RAW_ADC: now also R102.1 (A), U22.8 (D3); no longer R108.1 (A)
- net BUS_RAW_DIV_TOP: now also R91.2 (B), R92.1 (A); no longer R97.2 (B), R98.1 (A)
- net BUS_RAW_V_FILTER: now also D17.2 (A), D18.1 (K), R92.2 (B), R93.1 (A), C64.1 (A), U22.9 (S3); no longer D19.2 (A), D20.1 (K), R98.2 (B), R99.1 (A)
- net BUS_V_ADC: now also R100.1 (A), U22.3 (D1); no longer R106.1 (A)
- net BUS_V_FILTER: now also C62.1 (A), D13.2 (A), D14.1 (K), R86.2 (B), R87.1 (A), U22.2 (S1); no longer D15.2 (A), D16.1 (K), R92.2 (B), R93.1 (A)
- net CAP_DIV_TOP: now also R88.2 (B), R89.1 (A); no longer R94.2 (B), R95.1 (A)
- net CAP_I_ADC: now also R105.1 (A), U23.6 (D2)
- net CAP_I_FILTER: now also U23.5 (S2)
- net CAP_LINK: now also R88.1 (A); no longer R94.1 (A)
- net CAP_RAW_ADC: now also R103.1 (A), U22.11 (D4); no longer R109.1 (A)
- net CAP_RAW_DIV_TOP: now also R94.2 (B), R95.1 (A); no longer R100.2 (B), R101.1 (A)
- net CAP_RAW_V_FILTER: now also D19.2 (A), D20.1 (K), R95.2 (B), R96.1 (A), C65.1 (A), U22.12 (S4); no longer D21.2 (A), D22.1 (K), R101.2 (B), R102.1 (A)
- net CAP_V_ADC: now also R101.1 (A), U22.6 (D2); no longer R107.1 (A)
- net CAP_V_FILTER: now also D15.2 (A), D16.1 (K), C63.1 (A), R89.2 (B), R90.1 (A), U22.5 (S2); no longer D17.2 (A), D18.1 (K), R95.2 (B), R96.1 (A)
- net CLAMP_OR: now also D21.1 (K), D22.1 (K), R97.1 (A); no longer R103.1 (A)
- net CLAMP_REF: now also R98.2 (B), R99.1 (A), U21.1 (REF); no longer R104.2 (B), R105.1 (A)
- net GND: now also R100.2 (B), R101.2 (B), R103.2 (B), R104.2 (B), C62.2 (B), C63.2 (B), C64.2 (B), C65.2 (B), C66.2 (B), C67.2 (B), C68.2 (B), D14.2 (A), R87.2 (B), R90.2 (B), U21.3 (A), U22.7 (GND), U23.7 (GND), U24.12 (S4), U24.7 (GND), U24.9 (S3); no longer D22.2 (A)
- net IL_I_ADC: now also R106.1 (A), U23.8 (D3)
- net IL_I_FILTER: now also U23.9 (S3)
- net RAIL_OK: now also U22.1 (SEL1), U22.10 (SEL3), U22.13 (SEL4), U22.4 (SEL2), U23.1 (SEL1), U23.10 (SEL3), U23.13 (SEL4), U23.4 (SEL2), U24.1 (SEL1), U24.10 (SEL3), U24.13 (SEL4), U24.4 (SEL2)
- net TEMP_BANK_ADC: now also R109.1 (A), U24.6 (D2)
- net TEMP_BANK_FILTER: now also U24.5 (S2)
- net TEMP_FET_ADC: now also R107.1 (A), U23.11 (D4)
- net TEMP_FET_FILTER: now also U23.12 (S4)
- net TEMP_L_ADC: now also R108.1 (A), U24.3 (D1)
- net TEMP_L_FILTER: now also U24.2 (S1)
- net V3V3: now also C66.1 (A), C67.1 (A), C68.1 (A), U22.14 (VDD), U23.14 (VDD), U24.14 (VDD)
Other:
- moved on the sheet: D15, D16, D17, D18, D19, D20, D21, D22, R100, R101, R102, R103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
