File: hardware/kicad/robomaster_supercap.kicad_pcb (KiCad board)
At the start: 2 copper layers, 0 parts

Commit message: hardware: save Rev A placement and partial routing checkpoint
Parts:
- added C1: 470uF /63V EEUFR1J471 / ripple1.995Arms at100kHz, Capacitor_THT:CP_Radial_D12.5mm_P5.00mm, F.Cu at (30.0, 28.0)
- added C10: 470uF /63V EEUFR1J471 / ripple1.995Arms at100kHz, Capacitor_THT:CP_Radial_D12.5mm_P5.00mm, F.Cu at (94.0, 28.0)
- added C100: 100nF / 16V X7R, Capacitor_SMD:C_0805_2012Metric, F.Cu at (172.0, 125.0)
- added C101: 100nF / 16V X7R, Capacitor_SMD:C_0805_2012Metric, F.Cu at (172.0, 129.0)
- added C102: 100nF / 16V X7R, Capacitor_SMD:C_0805_2012Metric, F.Cu at (171.0, 133.0)
- added C103: 100nF / 16V X7R, Capacitor_SMD:C_0805_2012Metric, F.Cu at (177.0, 129.0)
- added C104: 100nF / 16V X7R, Capacitor_SMD:C_0805_2012Metric, F.Cu at (171.0, 106.0)
- added C105: 100nF / 16V X7R, Capacitor_SMD:C_0805_2012Metric, F.Cu at (176.0, 133.0)
- added C106: 100nF / 16V X7R, Capacitor_SMD:C_0805_2012Metric, F.Cu at (171.0, 137.0)
- added C107: 100nF / 16V X7R, Capacitor_SMD:C_0805_2012Metric, F.Cu at (182.0, 129.0)
- added C108: 100nF / 16V X7R, Capacitor_SMD:C_0805_2012Metric, F.Cu at (184.0, 125.0)
- added C109: 100nF / 16V X7R, Capacitor_SMD:C_0805_2012Metric, F.Cu at (145.0, 120.0)
- added C11: 470uF /63V EEUFR1J471 / ripple1.995Arms at100kHz, Capacitor_THT:CP_Radial_D12.5mm_P5.00mm, F.Cu at (108.0, 28.0)
- added C110: 100nF / 16V X7R, Capacitor_SMD:C_0805_2012Metric, F.Cu at (153.0, 136.0)
- added C111: 100nF / 16V X7R, Capacitor_SMD:C_0805_2012Metric, F.Cu at (185.0, 120.0)
- added C112: 100nF / 16V X7R, Capacitor_SMD:C_0805_2012Metric, F.Cu at (176.0, 137.0)
- added C113: 100nF / 16V X7R, Capacitor_SMD:C_0805_2012Metric, F.Cu at (145.0, 116.0)
- added C114: 100nF / 16V X7R, Capacitor_SMD:C_0805_2012Metric, F.Cu at (145.0, 124.0)
- added C115: 100nF / 16V X7R, Capacitor_SMD:C_0805_2012Metric, F.Cu at (146.0, 128.0)
- added C116: 100nF / 16V X7R, Capacitor_SMD:C_0805_2012Metric, F.Cu at (160.0, 140.0)
- added C117: 100nF / 16V X7R, Capacitor_SMD:C_0805_2012Metric, F.Cu at (181.0, 133.0)
- added C118: 100nF / 16V X7R, Capacitor_SMD:C_0805_2012Metric, F.Cu at (145.0, 112.0)
- added C119: 100nF / 16V X7R, Capacitor_SMD:C_0805_2012Metric, F.Cu at (170.0, 141.0)
- added C12: 470uF /63V EEUFR1J471 / ripple1.995Arms at100kHz, Capacitor_THT:CP_Radial_D12.5mm_P5.00mm, F.Cu at (80.0, 42.0)
- added C120: 100nF / 16V X7R, Capacitor_SMD:C_0805_2012Metric, F.Cu at (155.0, 140.0)
- added C121: 100nF / 16V X7R, Capacitor_SMD:C_0805_2012Metric, F.Cu at (146.0, 132.0)
- added C122: 100nF / 16V X7R, Capacitor_SMD:C_0805_2012Metric, F.Cu at (175.0, 141.0)
- added C123: 100nF / 16V X7R, Capacitor_SMD:C_0805_2012Metric, F.Cu at (145.0, 108.0)
- added C124: 100nF / 16V X7R, Capacitor_SMD:C_0805_2012Metric, F.Cu at (148.0, 136.0)
- added C125: 100nF / 16V X7R, Capacitor_SMD:C_0805_2012Metric, F.Cu at (181.0, 137.0)
- added C126: 100nF / 16V X7R, Capacitor_SMD:C_0805_2012Metric, F.Cu at (188.0, 116.0)
- added C127: 100nF / 16V X7R, Capacitor_SMD:C_0805_2012Metric, F.Cu at (187.0, 129.0)
- added C128: 100nF / 16V X7R, Capacitor_SMD:C_0805_2012Metric, F.Cu at (187.0, 110.0)
- added C129: 100nF / 16V X7R, Capacitor_SMD:C_0805_2012Metric, F.Cu at (189.0, 124.0)
- added C13: 470uF /63V EEUFR1J471 / ripple1.995Arms at100kHz, Capacitor_THT:CP_Radial_D12.5mm_P5.00mm, F.Cu at (94.0, 42.0)
- added C130: 1nF /50V, Capacitor_SMD:C_0805_2012Metric, F.Cu at (145.0, 104.0)
- added C131: 1nF /50V, Capacitor_SMD:C_0805_2012Metric, F.Cu at (145.0, 100.0)
- added C132: 1nF /50V, Capacitor_SMD:C_0805_2012Metric, F.Cu at (152.0, 92.0)
- added C133: 100nF / 16V X7R, Capacitor_SMD:C_0805_2012Metric, F.Cu at (160.0, 144.0)
- added C134: 100nF / 16V X7R, Capacitor_SMD:C_0805_2012Metric, F.Cu at (186.0, 133.0)
- added C135: 100nF / 16V X7R, Capacitor_SMD:C_0805_2012Metric, F.Cu at (140.0, 120.0)
- added C136: 100nF / 16V X7R, Capacitor_SMD:C_0805_2012Metric, F.Cu at (150.0, 140.0)
- added C137: 100nF / 16V X7R, Capacitor_SMD:C_0805_2012Metric, F.Cu at (190.0, 120.0)
- added C138: 100nF / 16V X7R, Capacitor_SMD:C_0805_2012Metric, F.Cu at (141.0, 128.0)
- added C139: 100nF / 16V X7R, Capacitor_SMD:C_0805_2012Metric, F.Cu at (140.0, 116.0)
- added C14: 470uF /63V EEUFR1J471 / ripple1.995Arms at100kHz, Capacitor_THT:CP_Radial_D12.5mm_P5.00mm, F.Cu at (108.0, 42.0)
- added C140: 100nF / 16V X7R, Capacitor_SMD:C_0805_2012Metric, F.Cu at (140.0, 124.0)
- added C15: 2.2uF / 100V X7R / effective C MUST VERIFY, Capacitor_SMD:C_1210_3225Metric, F.Cu at (92.0, 60.0)
- added C16: 2.2uF / 100V X7R / effective C MUST VERIFY, Capacitor_SMD:C_1210_3225Metric, F.Cu at (92.0, 84.0)
- added C17: 1nF /100V DNI tunable, Capacitor_SMD:C_0805_2012Metric, F.Cu at (70.0, 59.0)
- added C18: 1nF /100V DNI tunable, Capacitor_SMD:C_0805_2012Metric, F.Cu at (65.0, 59.0)
- added C19: 470nF /50V X7R bootstrap / effectiveC>=200nF target, Capacitor_SMD:C_0805_2012Metric, F.Cu at (47.0, 69.0)
- added C2: 470uF /63V EEUFR1J471 / ripple1.995Arms at100kHz, Capacitor_THT:CP_Radial_D12.5mm_P5.00mm, F.Cu at (44.0, 28.0)
- added C20: 1uF /25V X7R, Capacitor_SMD:C_0805_2012Metric, F.Cu at (49.5, 72.0)
- added C21: 100nF / 16V X7R, Capacitor_SMD:C_0805_2012Metric, F.Cu at (51.0, 75.0)
- added C22: 470nF /50V X7R bootstrap / effectiveC>=200nF target, Capacitor_SMD:C_0805_2012Metric, F.Cu at (87.0, 69.0)
- added C23: 1uF /25V X7R, Capacitor_SMD:C_0805_2012Metric, F.Cu at (89.5, 72.0)
- added C24: 100nF / 16V X7R, Capacitor_SMD:C_0805_2012Metric, F.Cu at (91.0, 75.0)
- added C25: 1nF EN filter, Capacitor_SMD:C_0805_2012Metric, F.Cu at (67.0, 114.0)
- added C26: 100nF / 16V X7R, Capacitor_SMD:C_0805_2012Metric, F.Cu at (73.0, 118.0)
- added C27: 100nF / 16V X7R, Capacitor_SMD:C_0805_2012Metric, F.Cu at (61.0, 126.0)
- added C28: 2.2nF /50V X7R mandatory, Capacitor_SMD:C_0805_2012Metric, F.Cu at (60.0, 176.0)
- added C29: 2.2uF /100V X7R, Capacitor_SMD:C_1210_3225Metric, F.Cu at (67.0, 163.0)
- added C3: 470uF /63V EEUFR1J471 / ripple1.995Arms at100kHz, Capacitor_THT:CP_Radial_D12.5mm_P5.00mm, F.Cu at (58.0, 28.0)
- added C30: 22uF /25V X7R, Capacitor_SMD:C_1210_3225Metric, F.Cu at (78.0, 187.0)
- added C31: 22uF /25V X7R, Capacitor_SMD:C_1210_3225Metric, F.Cu at (78.0, 192.0)
- added C32: 1nF C0G, Capacitor_SMD:C_0805_2012Metric, F.Cu at (57.0, 187.0)
- added C33: 100pF C0G, Capacitor_SMD:C_0805_2012Metric, F.Cu at (57.0, 183.0)
- added C34: 2.2nF /50V X7R mandatory, Capacitor_SMD:C_0805_2012Metric, F.Cu at (60.0, 169.0)
- added C35: 2.2uF /100V X7R, Capacitor_SMD:C_1210_3225Metric, F.Cu at (61.0, 163.0)
- added C36: 22uF /25V X7R, Capacitor_SMD:C_1210_3225Metric, F.Cu at (78.0, 182.0)
- added C37: 22uF /25V X7R, Capacitor_SMD:C_1210_3225Metric, F.Cu at (56.0, 192.0)
- added C38: 1nF C0G, Capacitor_SMD:C_0805_2012Metric, F.Cu at (74.0, 177.0)
- added C39: 100pF C0G, Capacitor_SMD:C_0805_2012Metric, F.Cu at (74.0, 173.0)
- added C4: 470uF /63V EEUFR1J471 / ripple1.995Arms at100kHz, Capacitor_THT:CP_Radial_D12.5mm_P5.00mm, F.Cu at (30.0, 42.0)
- added C40: 100nF / 16V X7R, Capacitor_SMD:C_0805_2012Metric, F.Cu at (200.0, 45.0)
- added C41: 100nF / 16V X7R, Capacitor_SMD:C_0805_2012Metric, F.Cu at (200.0, 41.0)
- added C42: 100nF / 16V X7R, Capacitor_SMD:C_0805_2012Metric, F.Cu at (200.0, 49.0)
- added C43: 100nF / 16V X7R, Capacitor_SMD:C_0805_2012Metric, F.Cu at (190.0, 55.0)
- added C44: 4.7uF /16V X7R, Capacitor_SMD:C_0805_2012Metric, F.Cu at (200.0, 37.0)
- added C45: 1uF /16V, Capacitor_SMD:C_0805_2012Metric, F.Cu at (185.0, 22.0)
- added C46: 100nF / 16V X7R, Capacitor_SMD:C_0805_2012Metric, F.Cu at (180.0, 22.0)
- added C47: 1uF /16V, Capacitor_SMD:C_0805_2012Metric, F.Cu at (185.0, 42.0)
- added C48: 100nF / 16V X7R, Capacitor_SMD:C_0805_2012Metric, F.Cu at (185.0, 46.0)
- added C49: 100nF, Capacitor_SMD:C_0805_2012Metric, F.Cu at (195.0, 32.0)
- added C5: 470uF /63V EEUFR1J471 / ripple1.995Arms at100kHz, Capacitor_THT:CP_Radial_D12.5mm_P5.00mm, F.Cu at (44.0, 42.0)
- added C50: 100nF / 16V X7R, Capacitor_SMD:C_0805_2012Metric, F.Cu at (152.0, 45.0)
- added C51: 1nF C0G, Capacitor_SMD:C_0805_2012Metric, F.Cu at (142.0, 45.0)
- added C52: 100nF / 16V X7R, Capacitor_SMD:C_0805_2012Metric, F.Cu at (152.0, 41.0)
- added C53: 100nF / 16V X7R, Capacitor_SMD:C_0805_2012Metric, F.Cu at (152.0, 49.0)
- added C54: 100nF / 16V X7R, Capacitor_SMD:C_0805_2012Metric, F.Cu at (142.0, 41.0)
- added C55: 1nF C0G, Capacitor_SMD:C_0805_2012Metric, F.Cu at (142.0, 49.0)
- added C56: 100nF / 16V X7R, Capacitor_SMD:C_0805_2012Metric, F.Cu at (152.0, 37.0)
- added C57: 100nF / 16V X7R, Capacitor_SMD:C_0805_2012Metric, F.Cu at (152.0, 53.0)
- added C58: 100nF / 16V X7R, Capacitor_SMD:C_0805_2012Metric, F.Cu at (157.0, 45.0)
- added C59: 1nF C0G, Capacitor_SMD:C_0805_2012Metric, F.Cu at (142.0, 37.0)
- added C6: 470uF /63V EEUFR1J471 / ripple1.995Arms at100kHz, Capacitor_THT:CP_Radial_D12.5mm_P5.00mm, F.Cu at (58.0, 42.0)
- added C60: 100nF / 16V X7R, Capacitor_SMD:C_0805_2012Metric, F.Cu at (142.0, 53.0)
- added C61: 100nF / 16V X7R, Capacitor_SMD:C_0805_2012Metric, F.Cu at (147.0, 35.0)
- added C62: 4.7nF C0G, Capacitor_SMD:C_0805_2012Metric, F.Cu at (252.0, 115.0)
- added C63: 4.7nF C0G, Capacitor_SMD:C_0805_2012Metric, F.Cu at (252.0, 135.0)
- added C64: 4.7nF C0G, Capacitor_SMD:C_0805_2012Metric, F.Cu at (246.0, 119.0)
- added C65: 4.7nF C0G, Capacitor_SMD:C_0805_2012Metric, F.Cu at (246.0, 139.0)
- added C66: 100nF / 16V X7R, Capacitor_SMD:C_0805_2012Metric, F.Cu at (265.0, 117.0)
- added C67: 100nF / 16V X7R, Capacitor_SMD:C_0805_2012Metric, F.Cu at (266.0, 113.0)
- added C68: 100nF / 16V X7R, Capacitor_SMD:C_0805_2012Metric, F.Cu at (267.0, 121.0)
- added C69: 10nF, Capacitor_SMD:C_0805_2012Metric, F.Cu at (235.0, 181.0)
- added C7: 2.2uF / 100V X7R / effective C MUST VERIFY, Capacitor_SMD:C_1210_3225Metric, F.Cu at (38.0, 60.0)
- added C70: 10nF, Capacitor_SMD:C_0805_2012Metric, F.Cu at (225.0, 187.0)
- added C71: 10nF, Capacitor_SMD:C_0805_2012Metric, F.Cu at (245.0, 187.0)
- added C8: 2.2uF / 100V X7R / effective C MUST VERIFY, Capacitor_SMD:C_1210_3225Metric, F.Cu at (38.0, 84.0)
- added C81: 100nF /50V X7R, Capacitor_SMD:C_0805_2012Metric, F.Cu at (278.0, 55.0)
- added C82: 100nF /50V X7R, Capacitor_SMD:C_0805_2012Metric, F.Cu at (278.0, 59.0)
- added C83: 100nF /50V X7R, Capacitor_SMD:C_0805_2012Metric, F.Cu at (278.0, 63.0)
- added C84: 100nF /50V X7R, Capacitor_SMD:C_0805_2012Metric, F.Cu at (278.0, 67.0)
- added C85: 100nF /50V X7R, Capacitor_SMD:C_0805_2012Metric, F.Cu at (278.0, 71.0)
- added C86: 100nF /50V X7R, Capacitor_SMD:C_0805_2012Metric, F.Cu at (273.0, 71.0)
- added C87: 100nF /50V X7R, Capacitor_SMD:C_0805_2012Metric, F.Cu at (273.0, 67.0)
- added C88: 100nF /50V X7R, Capacitor_SMD:C_0805_2012Metric, F.Cu at (273.0, 63.0)
- added C89: 100nF /50V X7R, Capacitor_SMD:C_0805_2012Metric, F.Cu at (273.0, 59.0)
- added C9: 470uF /63V EEUFR1J471 / ripple1.995Arms at100kHz, Capacitor_THT:CP_Radial_D12.5mm_P5.00mm, F.Cu at (80.0, 28.0)
- added C90: 100nF / 16V X7R, Capacitor_SMD:C_0805_2012Metric, F.Cu at (283.0, 33.0)
- added C91: 100nF / 16V X7R, Capacitor_SMD:C_0805_2012Metric, F.Cu at (283.0, 37.0)
- added C92: 100nF / 16V X7R, Capacitor_SMD:C_0805_2012Metric, F.Cu at (267.0, 53.0)
- added C93: 100nF / 16V X7R, Capacitor_SMD:C_0805_2012Metric, F.Cu at (255.0, 47.0)
- added C94: 100nF / 16V X7R, Capacitor_SMD:C_0805_2012Metric, F.Cu at (257.0, 53.0)
- added C95: 1uF /50V X7R, Capacitor_SMD:C_0805_2012Metric, F.Cu at (287.0, 47.0)
- added C96: 1uF /16V, Capacitor_SMD:C_0805_2012Metric, F.Cu at (273.0, 55.0)
- added C97: 1uF /16V, Capacitor_SMD:C_0805_2012Metric, F.Cu at (288.0, 37.0)
- added C98: 1uF /16V, Capacitor_SMD:C_0805_2012Metric, F.Cu at (283.0, 55.0)
- added C99: 100nF / 16V X7R, Capacitor_SMD:C_0805_2012Metric, F.Cu at (292.0, 185.0)
- added D1: SMBJ28A / no surge-energy guarantee, Diode_SMD:D_SMB, F.Cu at (56.0, 230.0)
- added D10: 1N4148W DNI turnoff bypass, Diode_SMD:D_SOD-123, F.Cu at (73.0, 122.0)
- added D11: 1N4148W DNI turnoff bypass, Diode_SMD:D_SOD-123, F.Cu at (61.0, 122.0)
- added D12: 1N4148W DNI turnoff bypass, Diode_SMD:D_SOD-123, F.Cu at (73.0, 126.0)
- added D13: BAT54H signal clamp, Diode_SMD:D_SOD-123F, F.Cu at (252.0, 123.0)
- added D14: BAT54H negative clamp, Diode_SMD:D_SOD-123F, F.Cu at (252.0, 119.0)
- added D15: BAT54H signal clamp, Diode_SMD:D_SOD-123F, F.Cu at (252.0, 127.0)
- added D16: BAT54H negative clamp, Diode_SMD:D_SOD-123F, F.Cu at (252.0, 131.0)
- added D17: BAT54H signal clamp, Diode_SMD:D_SOD-123F, F.Cu at (246.0, 127.0)
- added D18: BAT54H negative clamp, Diode_SMD:D_SOD-123F, F.Cu at (246.0, 123.0)
- added D19: BAT54H signal clamp, Diode_SMD:D_SOD-123F, F.Cu at (246.0, 131.0)
- added D2: SMBJ18CA bidirectional coil suppression / release MUST VERI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, Diode_SMD:D_SMB, F.Cu at (53.0, 224.0)
- added D20: BAT54H negative clamp, Diode_SMD:D_SOD-123F, F.Cu at (246.0, 135.0)
- added D21: 1N4148W /100V, Diode_SMD:D_SOD-123, F.Cu at (260.0, 112.0)
- added D22: 1N4148W /100V, Diode_SMD:D_SOD-123, F.Cu at (260.0, 108.0)
- added D23: SMBJ18CA bidirectional coil suppression / release MUST VERI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, Diode_SMD:D_SMB, F.Cu at (262.0, 59.0)
- added D24: BZT52H-C15, Diode_SMD:D_SOD-123F, F.Cu at (183.0, 197.0)
- added D25: red residual-energy indicator / bank-powered, LED_SMD:LED_0805_2012Metric, F.Cu at (197.0, 197.0)
- added D3: SMBJ18CA bidirectional coil suppression / release MUST VERI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, Diode_SMD:D_SMB, F.Cu at (142.0, 211.0)
- added D4: SMBJ18CA bidirectional coil suppression / release MUST VERI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, Diode_SMD:D_SMB, F.Cu at (142.0, 217.0)
- added D5: BZT52H-C15 / gate clamp candidate, Diode_SMD:D_SOD-123F, F.Cu at (34.5, 65.0)
- added D6: BZT52H-C15 / gate clamp candidate, Diode_SMD:D_SOD-123F, F.Cu at (34.5, 78.0)
- added D7: BZT52H-C15 / gate clamp candidate, Diode_SMD:D_SOD-123F, F.Cu at (74.5, 58.0)
- added D8: BZT52H-C15 / gate clamp candidate, Diode_SMD:D_SOD-123F, F.Cu at (74.5, 84.0)
- added D9: 1N4148W DNI turnoff bypass, Diode_SMD:D_SOD-123, F.Cu at (67.0, 126.0)
- added H1: MountingHole_3.2mm_M3, MountingHole_3.2mm_M3, F.Cu at (10.0, 10.0)
- added H2: MountingHole_3.2mm_M3, MountingHole_3.2mm_M3, F.Cu at (315.0, 10.0)
- added H3: MountingHole_3.2mm_M3, MountingHole_3.2mm_M3, F.Cu at (10.0, 235.0)
- added H4: MountingHole_3.2mm_M3, MountingHole_3.2mm_M3, F.Cu at (315.0, 235.0)
- added J10: L NTC probe option, Connector_PinHeader_2.54mm:PinHeader_1x02_P2.54mm_Vertical, F.Cu at (230.0, 187.0)
- added J11: BANK NTC probe option, Connector_PinHeader_2.54mm:PinHeader_1x02_P2.54mm_Vertical, F.Cu at (240.0, 187.0)
- added J17: selectable termination shunt, fit only at bus end, Connector_PinHeader_2.54mm:PinHeader_1x02_P2.54mm_Vertical, F.Cu at (287.0, 185.0)
- added J18: latched fault diagnostic output, Connector_PinHeader_2.54mm:PinHeader_1x02_P2.54mm_Vertical, F.Cu at (165.0, 120.0)
- added J19: ACTUATOR_12V / soldered harness with fixture strain relief, Connector_Wire:SolderWire-0.5sqmm_1x01_D0.9mm_OD2.1mm, F.Cu at (10.0, 18.0)
- added J20: BANK_P_RAW / soldered harness with fixture strain relief, Connector_Wire:SolderWire-0.5sqmm_1x01_D0.9mm_OD2.1mm, F.Cu at (10.0, 31.0)
- added J21: BUS_FUSED / soldered harness with fixture strain relief, Connector_Wire:SolderWire-2sqmm_1x01_D2mm_OD3.9mm, F.Cu at (10.0, 44.0)
- added J22: BUS_ISO_COIL_M / soldered harness with fixture strain relief, Connector_Wire:SolderWire-0.5sqmm_1x01_D0.9mm_OD2.1mm, F.Cu at (10.0, 57.0)
- added J23: BUS_ISO_FB / soldered harness with fixture strain relief, Connector_Wire:SolderWire-0.5sqmm_1x01_D0.9mm_OD2.1mm, F.Cu at (10.0, 70.0)
- added J24: BUS_LINK_IN / soldered harness with fixture strain relief, Connector_Wire:SolderWire-2sqmm_1x01_D2mm_OD3.9mm, F.Cu at (10.0, 83.0)
- added J25: BYP_BUS_COIL_M / soldered harness with fixture strain relief, Connector_Wire:SolderWire-0.5sqmm_1x01_D0.9mm_OD2.1mm, F.Cu at (10.0, 96.0)
- added J26: BYP_BUS_FB / soldered harness with fixture strain relief, Connector_Wire:SolderWire-0.5sqmm_1x01_D0.9mm_OD2.1mm, F.Cu at (10.0, 109.0)
- added J27: BYP_CAP_COIL_M / soldered harness with fixture strain relief, Connector_Wire:SolderWire-0.5sqmm_1x01_D0.9mm_OD2.1mm, F.Cu at (10.0, 122.0)
- added J28: BYP_CAP_FB / soldered harness with fixture strain relief, Connector_Wire:SolderWire-0.5sqmm_1x01_D0.9mm_OD2.1mm, F.Cu at (10.0, 135.0)
- added J29: CAN_H / soldered harness with fixture strain relief, Connector_Wire:SolderWire-0.5sqmm_1x01_D0.9mm_OD2.1mm, F.Cu at (10.0, 148.0)
- added J30: CAN_L / soldered harness with fixture strain relief, Connector_Wire:SolderWire-0.5sqmm_1x01_D0.9mm_OD2.1mm, F.Cu at (10.0, 161.0)
- added J31: CAP_ISO_COIL_M / soldered harness with fixture strain relief, Connector_Wire:SolderWire-0.5sqmm_1x01_D0.9mm_OD2.1mm, F.Cu at (10.0, 174.0)
- added J32: CAP_ISO_FB / soldered harness with fixture strain relief, Connector_Wire:SolderWire-0.5sqmm_1x01_D0.9mm_OD2.1mm, F.Cu at (10.0, 187.0)
- added J33: CAP_LINK_IN / soldered harness with fixture strain relief, Connector_Wire:SolderWire-2sqmm_1x01_D2mm_OD3.9mm, F.Cu at (10.0, 200.0)
- added J34: DUMP_DRAIN / soldered harness with fixture strain relief, Connector_Wire:SolderWire-0.5sqmm_1x01_D0.9mm_OD2.1mm, F.Cu at (10.0, 213.0)
- added J35: GND / soldered harness with fixture strain relief, Connector_Wire:SolderWire-2sqmm_1x01_D2mm_OD3.9mm, F.Cu at (315.0, 18.0)
- added J36: PRE_BUS_LED_M / soldered harness with fixture strain relief, Connector_Wire:SolderWire-0.5sqmm_1x01_D0.9mm_OD2.1mm, F.Cu at (315.0, 31.0)
- added J37: PRE_BUS_LED_P / soldered harness with fixture strain relief, Connector_Wire:SolderWire-0.5sqmm_1x01_D0.9mm_OD2.1mm, F.Cu at (315.0, 44.0)
- added J38: PRE_CAP_LED_M / soldered harness with fixture strain relief, Connector_Wire:SolderWire-0.5sqmm_1x01_D0.9mm_OD2.1mm, F.Cu at (315.0, 57.0)
- added J39: PRE_CAP_LED_P / soldered harness with fixture strain relief, Connector_Wire:SolderWire-0.5sqmm_1x01_D0.9mm_OD2.1mm, F.Cu at (315.0, 70.0)
- added J40: REFEREE_PERMIT / soldered harness with fixture strain relief, Connector_Wire:SolderWire-0.5sqmm_1x01_D0.9mm_OD2.1mm, F.Cu at (315.0, 83.0)
- added J41: TAP0_SOURCE_PROTECTED / soldered harness with fixture strai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, Connector_Wire:SolderWire-0.5sqmm_1x01_D0.9mm_OD2.1mm, F.Cu at (315.0, 96.0)
- added J42: TAP1_SOURCE_PROTECTED / soldered harness with fixture strai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, Connector_Wire:SolderWire-0.5sqmm_1x01_D0.9mm_OD2.1mm, F.Cu at (315.0, 109.0)
- added J43: TAP2_SOURCE_PROTECTED / soldered harness with fixture strai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, Connector_Wire:SolderWire-0.5sqmm_1x01_D0.9mm_OD2.1mm, F.Cu at (315.0, 122.0)
- added J44: TAP3_SOURCE_PROTECTED / soldered harness with fixture strai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, Connector_Wire:SolderWire-0.5sqmm_1x01_D0.9mm_OD2.1mm, F.Cu at (315.0, 135.0)
- added J45: TAP4_SOURCE_PROTECTED / soldered harness with fixture strai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, Connector_Wire:SolderWire-0.5sqmm_1x01_D0.9mm_OD2.1mm, F.Cu at (315.0, 148.0)
- added J46: TAP5_SOURCE_PROTECTED / soldered harness with fixture strai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, Connector_Wire:SolderWire-0.5sqmm_1x01_D0.9mm_OD2.1mm, F.Cu at (315.0, 161.0)
- added J47: TAP6_SOURCE_PROTECTED / soldered harness with fixture strai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, Connector_Wire:SolderWire-0.5sqmm_1x01_D0.9mm_OD2.1mm, F.Cu at (315.0, 174.0)
- added J48: TAP7_SOURCE_PROTECTED / soldered harness with fixture strai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, Connector_Wire:SolderWire-0.5sqmm_1x01_D0.9mm_OD2.1mm, F.Cu at (315.0, 187.0)
- added J49: TAP8_SOURCE_PROTECTED / soldered harness with fixture strai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, Connector_Wire:SolderWire-0.5sqmm_1x01_D0.9mm_OD2.1mm, F.Cu at (315.0, 200.0)
- added J50: TAP9_SOURCE_PROTECTED / soldered harness with fixture strai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, Connector_Wire:SolderWire-0.5sqmm_1x01_D0.9mm_OD2.1mm, F.Cu at (315.0, 213.0)
- added J6: SWD reference voltage ONLY / do not externally power, Connector_PinHeader_2.54mm:PinHeader_1x06_P2.54mm_Vertical, F.Cu at (195.0, 45.0)
- added J7: 3.3V UART / no power pin, Connector_PinHeader_2.54mm:PinHeader_1x03_P2.54mm_Vertical, F.Cu at (190.0, 45.0)
- added J8: OC diagnostic outputs / do not load, Connector_PinHeader_2.54mm:PinHeader_1x05_P2.54mm_Vertical, F.Cu at (147.0, 45.0)
- added J9: FET NTC probe option, Connector_PinHeader_2.54mm:PinHeader_1x02_P2.54mm_Vertical, F.Cu at (235.0, 187.0)
- added L1: XAL1510-223MED / 22uH +/-20%, Inductor_SMD:L_Coilcraft_XAL1510-223, F.Cu at (65.0, 70.0)
- added L2: 68uH / MSS1246T-683MLB, Inductor_SMD:L_Coilcraft_MSS1246T-XXX, F.Cu at (67.0, 187.0)
- added L3: 47uH / MSS1246T-473MLB, Inductor_SMD:L_Coilcraft_MSS1246T-XXX, F.Cu at (67.0, 201.0)
- added Q1: CSD18540Q5B, Package_SON:VSONP-8-1EP_5x6_P1.27mm, F.Cu at (65.0, 230.0)
- added Q10: BC857B, Package_TO_SOT_SMD:SOT-23, F.Cu at (142.0, 205.0)
- added Q11: BC847B, Package_TO_SOT_SMD:SOT-23, F.Cu at (136.0, 200.0)
- added Q12: CSD18540Q5B, Package_SON:VSONP-8-1EP_5x6_P1.27mm, F.Cu at (45.0, 65.0)
- added Q13: CSD18540Q5B, Package_SON:VSONP-8-1EP_5x6_P1.27mm, F.Cu at (45.0, 78.0)
- added Q14: CSD18540Q5B, Package_SON:VSONP-8-1EP_5x6_P1.27mm, F.Cu at (85.0, 65.0)
- added Q15: CSD18540Q5B, Package_SON:VSONP-8-1EP_5x6_P1.27mm, F.Cu at (85.0, 78.0)
- added Q16: CSD18540Q5B, Package_SON:VSONP-8-1EP_5x6_P1.27mm, F.Cu at (262.0, 47.0)
- added Q17: BC857B, Package_TO_SOT_SMD:SOT-23, F.Cu at (262.0, 53.0)
- added Q18: BC847B, Package_TO_SOT_SMD:SOT-23, F.Cu at (262.0, 41.0)
- added Q19: BC847B preregulator / voltage thermal MUST VERIFY, Package_TO_SOT_SMD:SOT-23, F.Cu at (269.0, 47.0)
- added Q2: BC857B, Package_TO_SOT_SMD:SOT-23, F.Cu at (65.0, 224.0)
- added Q20: CSD18540Q5B, Package_SON:VSONP-8-1EP_5x6_P1.27mm, F.Cu at (190.0, 197.0)
- added Q21: BC857B, Package_TO_SOT_SMD:SOT-23, F.Cu at (190.0, 203.0)
- added Q22: BC847B, Package_TO_SOT_SMD:SOT-23, F.Cu at (190.0, 191.0)
- added Q3: BC847B, Package_TO_SOT_SMD:SOT-23, F.Cu at (65.0, 236.0)
- added Q4: BC847B, Package_TO_SOT_SMD:SOT-23, F.Cu at (142.0, 195.0)
- added Q5: CSD18540Q5B, Package_SON:VSONP-8-1EP_5x6_P1.27mm, F.Cu at (142.0, 189.0)
- added Q6: BC857B, Package_TO_SOT_SMD:SOT-23, F.Cu at (142.0, 200.0)
- added Q7: BC847B, Package_TO_SOT_SMD:SOT-23, F.Cu at (148.0, 195.0)
- added Q8: BC847B, Package_TO_SOT_SMD:SOT-23, F.Cu at (136.0, 195.0)
- added Q9: CSD18540Q5B, Package_SON:VSONP-8-1EP_5x6_P1.27mm, F.Cu at (149.0, 201.0)
- added R1: 10k, Resistor_SMD:R_0805_2012Metric, F.Cu at (72.0, 230.0)
- added R10: 1.5k, Resistor_SMD:R_0805_2012Metric, F.Cu at (135.0, 190.0)
- added R100: 100k off leakage drain, Resistor_SMD:R_0805_2012Metric, F.Cu at (267.0, 125.0)
- added R101: 100k off leakage drain, Resistor_SMD:R_0805_2012Metric, F.Cu at (267.0, 129.0)
- added R102: 100k off leakage drain, Resistor_SMD:R_0805_2012Metric, F.Cu at (272.0, 123.0)
- added R103: 100k off leakage drain, Resistor_SMD:R_0805_2012Metric, F.Cu at (267.0, 133.0)
- added R104: 100k off leakage drain, Resistor_SMD:R_0805_2012Metric, F.Cu at (267.0, 137.0)
- added R105: 100k off leakage drain, Resistor_SMD:R_0805_2012Metric, F.Cu at (253.0, 139.0)
- added R106: 100k off leakage drain, Resistor_SMD:R_0805_2012Metric, F.Cu at (272.0, 130.0)
- added R107: 100k off leakage drain, Resistor_SMD:R_0805_2012Metric, F.Cu at (272.0, 134.0)
- added R108: 100k off leakage drain, Resistor_SMD:R_0805_2012Metric, F.Cu at (260.0, 143.0)
- added R109: 100k off leakage drain, Resistor_SMD:R_0805_2012Metric, F.Cu at (255.0, 143.0)
- added R11: 10k, Resistor_SMD:R_0805_2012Metric, F.Cu at (135.0, 186.0)
- added R110: 10k /1%, Resistor_SMD:R_0805_2012Metric, F.Cu at (235.0, 177.0)
- added R111: NTCLE100E3103JB0 /10k NTC B3977, Connector_PinHeader_2.54mm:PinHeader_1x02_P2.54mm_Vertical, F.Cu at (230.0, 177.0)
- added R112: 10k /1%, Resistor_SMD:R_0805_2012Metric, F.Cu at (225.0, 183.0)
- added R113: NTCLE100E3103JB0 /10k NTC B3977, Connector_PinHeader_2.54mm:PinHeader_1x02_P2.54mm_Vertical, F.Cu at (220.0, 183.0)
- added R114: 10k /1%, Resistor_SMD:R_0805_2012Metric, F.Cu at (245.0, 183.0)
- added R115: NTCLE100E3103JB0 /10k NTC B3977, Connector_PinHeader_2.54mm:PinHeader_1x02_P2.54mm_Vertical, F.Cu at (250.0, 183.0)
- added R116: 10k, Resistor_SMD:R_0805_2012Metric, F.Cu at (257.0, 41.0)
- added R117: 10k, Resistor_SMD:R_0805_2012Metric, F.Cu at (262.0, 64.0)
- added R118: 10k, Resistor_SMD:R_0805_2012Metric, F.Cu at (262.0, 68.0)
- added R119: 4.7k, Resistor_SMD:R_0805_2012Metric, F.Cu at (262.0, 36.0)
- added R12: 10k, Resistor_SMD:R_0805_2012Metric, F.Cu at (153.0, 195.0)
- added R120: 100k, Resistor_SMD:R_0805_2012Metric, F.Cu at (262.0, 32.0)
- added R121: 47R, Resistor_SMD:R_0805_2012Metric, F.Cu at (257.0, 37.0)
- added R122: 10k, Resistor_SMD:R_0805_2012Metric, F.Cu at (267.0, 41.0)
- added R133: 1k /1W tap protection / no bypass, Resistor_SMD:R_2512_6332Metric, F.Cu at (285.0, 60.0)
- added R134: 1k /1W tap protection / no bypass, Resistor_SMD:R_2512_6332Metric, F.Cu at (285.0, 66.0)
- added R135: 1k /1W tap protection / no bypass, Resistor_SMD:R_2512_6332Metric, F.Cu at (285.0, 72.0)
- added R136: 1k /1W tap protection / no bypass, Resistor_SMD:R_2512_6332Metric, F.Cu at (294.0, 67.0)
- added R137: 1k /1W tap protection / no bypass, Resistor_SMD:R_2512_6332Metric, F.Cu at (294.0, 61.0)
- added R138: 1k /1W tap protection / no bypass, Resistor_SMD:R_2512_6332Metric, F.Cu at (255.0, 71.0)
- added R139: 1k /1W tap protection / no bypass, Resistor_SMD:R_2512_6332Metric, F.Cu at (255.0, 65.0)
- added R14: 10k, Resistor_SMD:R_0805_2012Metric, F.Cu at (142.0, 183.0)
- added R140: 1k /1W tap protection / no bypass, Resistor_SMD:R_2512_6332Metric, F.Cu at (290.0, 54.0)
- added R141: 1k /1W tap protection / no bypass, Resistor_SMD:R_2512_6332Metric, F.Cu at (253.0, 59.0)
- added R142: 1k /1W tap protection / no bypass, Resistor_SMD:R_2512_6332Metric, F.Cu at (289.0, 42.0)
- added R143: 10k, Resistor_SMD:R_0805_2012Metric, F.Cu at (284.0, 29.0)
- added R144: 10k, Resistor_SMD:R_0805_2012Metric, F.Cu at (288.0, 33.0)
- added R145: 10k, Resistor_SMD:R_0805_2012Metric, F.Cu at (289.0, 29.0)
- added R146: 10k, Resistor_SMD:R_0805_2012Metric, F.Cu at (270.0, 22.0)
- added R147: 10k, Resistor_SMD:R_0805_2012Metric, F.Cu at (263.0, 28.0)
- added R148: 100R, Resistor_SMD:R_0805_2012Metric, F.Cu at (292.0, 47.0)
- added R149: 0R, Resistor_SMD:R_0805_2012Metric, F.Cu at (297.0, 47.0)
- added R15: 10k, Resistor_SMD:R_0805_2012Metric, F.Cu at (142.0, 222.0)
- added R150: 10k, Resistor_SMD:R_0805_2012Metric, F.Cu at (296.0, 43.0)
- added R151: 10k, Resistor_SMD:R_0805_2012Metric, F.Cu at (296.0, 39.0)
- added R152: 10k TS commissioning option, Resistor_SMD:R_0805_2012Metric, F.Cu at (293.0, 35.0)
- added R153: 10k TS commissioning option, Resistor_SMD:R_0805_2012Metric, F.Cu at (297.0, 51.0)
- added R154: 10k TS commissioning option, Resistor_SMD:R_0805_2012Metric, F.Cu at (268.0, 64.0)
- added R155: 10k, Resistor_SMD:R_0805_2012Metric, F.Cu at (297.0, 55.0)
- added R156: 10k, Resistor_SMD:R_0805_2012Metric, F.Cu at (294.0, 31.0)
- added R157: 10k /1W permanent bleed, Resistor_SMD:R_2512_6332Metric, F.Cu at (182.0, 203.0)
- added R159: 10k, Resistor_SMD:R_0805_2012Metric, F.Cu at (183.0, 193.0)
- added R16: 10k, Resistor_SMD:R_0805_2012Metric, F.Cu at (137.0, 222.0)
- added R160: 47R, Resistor_SMD:R_0805_2012Metric, F.Cu at (183.0, 189.0)
- added R161: 10k, Resistor_SMD:R_0805_2012Metric, F.Cu at (190.0, 208.0)
- added R162: 10k, Resistor_SMD:R_0805_2012Metric, F.Cu at (190.0, 212.0)
- added R163: 4.7k, Resistor_SMD:R_0805_2012Metric, F.Cu at (190.0, 186.0)
- added R164: 100k, Resistor_SMD:R_0805_2012Metric, F.Cu at (190.0, 182.0)
- added R165: 22k /0.25W, Resistor_SMD:R_0805_2012Metric, F.Cu at (182.0, 208.0)
- added R167: 10k, Resistor_SMD:R_0805_2012Metric, F.Cu at (280.0, 179.0)
- added R168: 10k, Resistor_SMD:R_0805_2012Metric, F.Cu at (280.0, 191.0)
- added R169: 120R /1%, Resistor_SMD:R_0805_2012Metric, F.Cu at (273.0, 185.0)
- added R17: 4.7k, Resistor_SMD:R_0805_2012Metric, F.Cu at (154.0, 191.0)
- added R170: 58.7k /1%, Resistor_SMD:R_0805_2012Metric, F.Cu at (140.0, 112.0)
- added R171: 10k /PROVISIONAL, Resistor_SMD:R_0805_2012Metric, F.Cu at (140.0, 108.0)
- added R172: 35.7k /1%, Resistor_SMD:R_0805_2012Metric, F.Cu at (180.0, 98.0)
- added R173: 10k /PROVISIONAL, Resistor_SMD:R_0805_2012Metric, F.Cu at (180.0, 94.0)
- added R174: 35.7k, Resistor_SMD:R_0805_2012Metric, F.Cu at (170.0, 145.0)
- added R175: 10k / IL12.035A PROVISIONAL, Resistor_SMD:R_0805_2012Metric, F.Cu at (170.0, 149.0)
- added R176: 10k, Resistor_SMD:R_0805_2012Metric, F.Cu at (155.0, 144.0)
- added R177: 10k / preset timeout; verify SET1 table, Resistor_SMD:R_0805_2012Metric, F.Cu at (187.0, 106.0)
- added R178: 10k, Resistor_SMD:R_0805_2012Metric, F.Cu at (141.0, 132.0)
- added R179: 10k, Resistor_SMD:R_0805_2012Metric, F.Cu at (143.0, 136.0)
- added R18: 100k, Resistor_SMD:R_0805_2012Metric, F.Cu at (154.0, 187.0)
- added R180: 10k, Resistor_SMD:R_0805_2012Metric, F.Cu at (135.0, 116.0)
- added R181: 10k, Resistor_SMD:R_0805_2012Metric, F.Cu at (140.0, 104.0)
- added R182: 10k, Resistor_SMD:R_0805_2012Metric, F.Cu at (145.0, 96.0)
- added R183: 10k, Resistor_SMD:R_0805_2012Metric, F.Cu at (140.0, 100.0)
- added R184: 10k, Resistor_SMD:R_0805_2012Metric, F.Cu at (147.0, 92.0)
- added R185: 10k, Resistor_SMD:R_0805_2012Metric, F.Cu at (151.0, 88.0)
- added R186: 10k, Resistor_SMD:R_0805_2012Metric, F.Cu at (187.0, 102.0)
- added R187: 1.74k /PROVISIONAL, Resistor_SMD:R_0805_2012Metric, F.Cu at (187.0, 98.0)
- added R188: 10k, Resistor_SMD:R_0805_2012Metric, F.Cu at (193.0, 116.0)
- added R189: 1.74k /PROVISIONAL, Resistor_SMD:R_0805_2012Metric, F.Cu at (193.0, 112.0)
- added R19: 47R, Resistor_SMD:R_0805_2012Metric, F.Cu at (142.0, 179.0)
- added R190: 10k, Resistor_SMD:R_0805_2012Metric, F.Cu at (192.0, 108.0)
- added R191: 3.01k /PROVISIONAL, Resistor_SMD:R_0805_2012Metric, F.Cu at (192.0, 104.0)
- added R192: 1k, Resistor_SMD:R_0805_2012Metric, F.Cu at (195.0, 120.0)
- added R193: 10k, Resistor_SMD:R_0805_2012Metric, F.Cu at (195.0, 124.0)
- added R194: 2.2k, Resistor_SMD:R_0805_2012Metric, F.Cu at (173.0, 89.0)
- added R195: 221k /1%, Resistor_SMD:R_0805_2012Metric, F.Cu at (140.0, 96.0)
- added R196: 10k /1%, Resistor_SMD:R_0805_2012Metric, F.Cu at (140.0, 92.0)
- added R197: 154k /1%, Resistor_SMD:R_0805_2012Metric, F.Cu at (135.0, 96.0)
- added R198: 10k /1%, Resistor_SMD:R_0805_2012Metric, F.Cu at (135.0, 92.0)
- added R199: 172k /1%, Resistor_SMD:R_0805_2012Metric, F.Cu at (157.0, 90.0)
- added R2: 10k, Resistor_SMD:R_0805_2012Metric, F.Cu at (60.0, 224.0)
- added R20: 10k, Resistor_SMD:R_0805_2012Metric, F.Cu at (149.0, 186.0)
- added R200: 10k /1%, Resistor_SMD:R_0805_2012Metric, F.Cu at (157.0, 86.0)
- added R201: 80.6k, Resistor_SMD:R_0805_2012Metric, F.Cu at (165.0, 89.0)
- added R202: 10k, Resistor_SMD:R_0805_2012Metric, F.Cu at (165.0, 85.0)
- added R203: 100k, Resistor_SMD:R_0805_2012Metric, F.Cu at (170.0, 85.0)
- added R204: 10k, Resistor_SMD:R_0805_2012Metric, F.Cu at (175.0, 85.0)
- added R205: 78.7k, Resistor_SMD:R_0805_2012Metric, F.Cu at (179.0, 90.0)
- added R206: 10k, Resistor_SMD:R_0805_2012Metric, F.Cu at (180.0, 86.0)
- added R207: 100k, Resistor_SMD:R_0805_2012Metric, F.Cu at (184.0, 90.0)
- added R208: 10k, Resistor_SMD:R_0805_2012Metric, F.Cu at (185.0, 86.0)
- added R21: 150R, Resistor_SMD:R_0805_2012Metric, F.Cu at (137.0, 205.0)
- added R22: 1.5k, Resistor_SMD:R_0805_2012Metric, F.Cu at (131.0, 195.0)
- added R23: 10k, Resistor_SMD:R_0805_2012Metric, F.Cu at (131.0, 199.0)
- added R24: 10k, Resistor_SMD:R_0805_2012Metric, F.Cu at (130.0, 191.0)
- added R26: 10k, Resistor_SMD:R_0805_2012Metric, F.Cu at (149.0, 207.0)
- added R27: 10k, Resistor_SMD:R_0805_2012Metric, F.Cu at (147.0, 222.0)
- added R28: 10k, Resistor_SMD:R_0805_2012Metric, F.Cu at (149.0, 218.0)
- added R29: 4.7k, Resistor_SMD:R_0805_2012Metric, F.Cu at (131.0, 203.0)
- added R3: 10k, Resistor_SMD:R_0805_2012Metric, F.Cu at (70.0, 224.0)
- added R30: 100k, Resistor_SMD:R_0805_2012Metric, F.Cu at (131.0, 207.0)
- added R31: 47R, Resistor_SMD:R_0805_2012Metric, F.Cu at (149.0, 211.0)
- added R32: 10k, Resistor_SMD:R_0805_2012Metric, F.Cu at (147.0, 182.0)
- added R33: WSK25123L000FEA / 3mR 1% 1W, Resistor_SMD:R_Shunt_Vishay_WSK2512_6332Metric_T2.21mm, F.Cu at (30.0, 57.0)
- added R34: WSK25123L000FEA / 3mR 1% 1W, Resistor_SMD:R_Shunt_Vishay_WSK2512_6332Metric_T2.21mm, F.Cu at (108.0, 57.0)
- added R35: WSK25123L000FEA / 3mR 1% 1W, Resistor_SMD:R_Shunt_Vishay_WSK2512_6332Metric_T2.21mm, F.Cu at (55.0, 59.0)
- added R36: 10k GS mandatory, Resistor_SMD:R_0805_2012Metric, F.Cu at (39.0, 65.0)
- added R37: 10k GS mandatory, Resistor_SMD:R_0805_2012Metric, F.Cu at (39.0, 78.0)
- added R38: 10k GS mandatory, Resistor_SMD:R_0805_2012Metric, F.Cu at (79.0, 65.0)
- added R39: 10k GS mandatory, Resistor_SMD:R_0805_2012Metric, F.Cu at (79.0, 78.0)
- added R4: 4.7k, Resistor_SMD:R_0805_2012Metric, F.Cu at (60.0, 236.0)
- added R40: 10R DNI tunable, Resistor_SMD:R_0805_2012Metric, F.Cu at (70.0, 55.0)
- added R41: 10R DNI tunable, Resistor_SMD:R_0805_2012Metric, F.Cu at (65.0, 55.0)
- added R42: 4.7R gate / tunable, Resistor_SMD:R_0603_1608Metric, F.Cu at (39.0, 68.0)
- added R43: 2.2R DNI turnoff option, Resistor_SMD:R_0805_2012Metric, F.Cu at (67.0, 130.0)
- added R44: 4.7R gate / tunable, Resistor_SMD:R_0603_1608Metric, F.Cu at (39.0, 81.0)
- added R45: 2.2R DNI turnoff option, Resistor_SMD:R_0805_2012Metric, F.Cu at (79.0, 122.0)
- added R46: 10k, Resistor_SMD:R_0805_2012Metric, F.Cu at (61.0, 118.0)
- added R47: 10k, Resistor_SMD:R_0805_2012Metric, F.Cu at (62.0, 114.0)
- added R48: 4.7R gate / tunable, Resistor_SMD:R_0603_1608Metric, F.Cu at (79.0, 68.0)
- added R49: 2.2R DNI turnoff option, Resistor_SMD:R_0805_2012Metric, F.Cu at (55.0, 122.0)
- added R5: 100k, Resistor_SMD:R_0805_2012Metric, F.Cu at (55.0, 236.0)
- added R50: 4.7R gate / tunable, Resistor_SMD:R_0603_1608Metric, F.Cu at (79.0, 81.0)
- added R51: 2.2R DNI turnoff option, Resistor_SMD:R_0805_2012Metric, F.Cu at (73.0, 130.0)
- added R52: 10k, Resistor_SMD:R_0805_2012Metric, F.Cu at (72.0, 114.0)
- added R53: 10k, Resistor_SMD:R_0805_2012Metric, F.Cu at (67.0, 110.0)
- added R54: 10k, Resistor_SMD:R_0805_2012Metric, F.Cu at (62.0, 110.0)
- added R55: 909k, Resistor_SMD:R_0805_2012Metric, F.Cu at (55.0, 179.0)
- added R56: 100k, Resistor_SMD:R_0805_2012Metric, F.Cu at (55.0, 175.0)
- added R57: 100k, Resistor_SMD:R_0805_2012Metric, F.Cu at (74.0, 169.0)
- added R58: 1M, Resistor_SMD:R_0805_2012Metric, F.Cu at (55.0, 163.0)
- added R59: 82.5k, Resistor_SMD:R_0805_2012Metric, F.Cu at (55.0, 167.0)
- added R6: 47R, Resistor_SMD:R_0805_2012Metric, F.Cu at (72.0, 234.0)
- added R60: 10k, Resistor_SMD:R_0805_2012Metric, F.Cu at (79.0, 176.0)
- added R61: 1M, Resistor_SMD:R_0805_2012Metric, F.Cu at (52.0, 183.0)
- added R62: 174k, Resistor_SMD:R_0805_2012Metric, F.Cu at (79.0, 172.0)
- added R63: 100k, Resistor_SMD:R_0805_2012Metric, F.Cu at (79.0, 168.0)
- added R64: 27.4k, Resistor_SMD:R_0805_2012Metric, F.Cu at (74.0, 165.0)
- added R65: 1M, Resistor_SMD:R_0805_2012Metric, F.Cu at (50.0, 163.0)
- added R66: 82.5k, Resistor_SMD:R_0805_2012Metric, F.Cu at (50.0, 167.0)
- added R67: 10k, Resistor_SMD:R_0805_2012Metric, F.Cu at (55.0, 171.0)
- added R68: 475k, Resistor_SMD:R_0805_2012Metric, F.Cu at (84.0, 173.0)
- added R69: 10R, Resistor_SMD:R_0805_2012Metric, F.Cu at (190.0, 22.0)
- added R7: 10k, Resistor_SMD:R_0805_2012Metric, F.Cu at (70.0, 238.0)
- added R70: 0R, Resistor_SMD:R_0805_2012Metric, F.Cu at (195.0, 22.0)
- added R71: 10k, Resistor_SMD:R_0805_2012Metric, F.Cu at (195.0, 28.0)
- added R72: 10k, Resistor_SMD:R_0805_2012Metric, F.Cu at (180.0, 42.0)
- added R73: 10k, Resistor_SMD:R_0805_2012Metric, F.Cu at (180.0, 46.0)
- added R74: 10k, Resistor_SMD:R_0805_2012Metric, F.Cu at (200.0, 32.0)
- added R75: 10k, Resistor_SMD:R_0805_2012Metric, F.Cu at (200.0, 28.0)
- added R76: 10k, Resistor_SMD:R_0805_2012Metric, F.Cu at (200.0, 24.0)
- added R77: 10k, Resistor_SMD:R_0805_2012Metric, F.Cu at (185.0, 50.0)
- added R78: 10k, Resistor_SMD:R_0805_2012Metric, F.Cu at (180.0, 50.0)
- added R79: 10k, Resistor_SMD:R_0805_2012Metric, F.Cu at (205.0, 32.0)
- added R8: 10k, Resistor_SMD:R_0805_2012Metric, F.Cu at (75.0, 226.0)
- added R80: 10k, Resistor_SMD:R_0805_2012Metric, F.Cu at (205.0, 28.0)
- added R81: 10k, Resistor_SMD:R_0805_2012Metric, F.Cu at (205.0, 36.0)
- added R82: 100R, Resistor_SMD:R_0805_2012Metric, F.Cu at (137.0, 45.0)
- added R83: 100R, Resistor_SMD:R_0805_2012Metric, F.Cu at (137.0, 49.0)
- added R84: 100R, Resistor_SMD:R_0805_2012Metric, F.Cu at (142.0, 33.0)
- added R85: 33k /1%, Resistor_SMD:R_0805_2012Metric, F.Cu at (254.0, 111.0)
- added R86: 33k /1%, Resistor_SMD:R_0805_2012Metric, F.Cu at (254.0, 107.0)
- added R87: 5.1k /1%, Resistor_SMD:R_0805_2012Metric, F.Cu at (254.0, 103.0)
- added R88: 33k /1%, Resistor_SMD:R_0805_2012Metric, F.Cu at (270.0, 117.0)
- added R89: 33k /1%, Resistor_SMD:R_0805_2012Metric, F.Cu at (271.0, 113.0)
- added R9: 150R, Resistor_SMD:R_0805_2012Metric, F.Cu at (149.0, 190.0)
- added R90: 6.8k /1%, Resistor_SMD:R_0805_2012Metric, F.Cu at (271.0, 109.0)
- added R91: 33k /1%, Resistor_SMD:R_0805_2012Metric, F.Cu at (266.0, 109.0)
- added R92: 33k /1%, Resistor_SMD:R_0805_2012Metric, F.Cu at (266.0, 105.0)
- added R93: 5.1k /1%, Resistor_SMD:R_0805_2012Metric, F.Cu at (266.0, 101.0)
- added R94: 33k /1%, Resistor_SMD:R_0805_2012Metric, F.Cu at (260.0, 104.0)
- added R95: 33k /1%, Resistor_SMD:R_0805_2012Metric, F.Cu at (260.0, 100.0)
- added R96: 6.8k /1%, Resistor_SMD:R_0805_2012Metric, F.Cu at (260.0, 96.0)
- added R97: 3.3k /1W, Resistor_SMD:R_2512_6332Metric, F.Cu at (253.0, 98.0)
- added R98: 11.8k /1%, Resistor_SMD:R_0805_2012Metric, F.Cu at (253.0, 93.0)
- added R99: 10k /1%, Resistor_SMD:R_0805_2012Metric, F.Cu at (253.0, 89.0)
- added U10: LM5164DDAR, Package_SO:TI_SO-PowerPAD-8, F.Cu at (67.0, 169.0)
- added U11: STM32G474RET6, Package_QFP:LQFP-64_10x10mm_P0.5mm, F.Cu at (185.0, 32.0)
- added U12: INA240A2D, Package_SO:SOIC-8_3.9x4.9mm_P1.27mm, F.Cu at (27.0, 70.0)
- added U13: INA293A1DBVR, Package_TO_SOT_SMD:SOT-23-5, F.Cu at (27.0, 76.0)
- added U14: INA293A1DBVR, Package_TO_SOT_SMD:SOT-23-5, F.Cu at (27.0, 80.0)
- added U15: INA240A1D, Package_SO:SOIC-8_3.9x4.9mm_P1.27mm, F.Cu at (109.0, 70.0)
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Routing:
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- added copper zone on F.Cu, net GND
- added copper zone on In1.Cu, net GND
Other:
- board outline added: 315 x 235 mm
- copper layers 2 -> 4
- board text added: "REV A BENCH PROTOTYPE / NOT RELEASED"

Commit message: hardware: connect Rev A power paths and add ground fanout
Parts:
- moved J33 216.3 mm to (117.0, 12.0)
- moved R85 213.4 mm to (61.0, 20.0)
- moved R88 186.3 mm to (111.0, 20.0)
- moved J24 31.4 mm to (15.0, 52.0)
Routing:
- net GND: track 38.0 -> 302.7 mm, vias 24 -> 303
- net BUS_LINK: track 5.02 -> 193.9 mm, vias 0 -> 32
- net CAP_LINK: track 17.5 -> 191.8 mm, vias 0 -> 32
- net BUS_FUSED: track 158.0 -> 4.68 mm, vias 1 -> 0
- net BUS_FAST_NEG: track 214.1 -> 78.9 mm, vias 3 -> 1
- net SW_NODE_B: track 0.00 -> 102.0 mm, vias 0 -> 30
- net CAP_ISO_FB: track 0.00 -> 93.2 mm, vias 0 -> 3
- net SW_NODE_A: track 18.6 -> 97.1 mm, vias 2 -> 23
- net HO_B: track 66.0 -> 0.00 mm, vias 4 -> 0
- net CAP_LINK_IN: track 0.00 -> 63.6 mm, vias 0 -> 6
- net MON_SCLK: track 0.00 -> 34.4 mm, vias 0 -> 3
- net BUS_KELVIN_M: track 31.3 -> 0.00 mm, vias 2 -> 0
- net IL_KELVIN_M: track 29.3 -> 0.00 mm, vias 2 -> 0
- net NRST: track 16.3 -> 41.7 mm, vias 0 -> 1
- net MON_LD: track 0.00 -> 23.3 mm, vias 0 -> 2
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
Commit message: hardware: complete Prototype Rev A PCB routing and validation
Parts:
- moved R43 67.4 mm to (34.5, 71.0), turned to 180 degrees
- moved D9 66.5 mm to (34.5, 68.0)
- moved R49 62.5 mm to (75.5, 63.0), turned to 180 degrees
- moved R45 59.7 mm to (33.0, 84.0), turned to 180 degrees
- moved R51 57.1 mm to (75.5, 73.0), turned to 180 degrees
- moved D10 56.2 mm to (34.5, 81.0)
- moved D11 55.9 mm to (75.5, 68.0), turned to 90 degrees
- moved D12 48.1 mm to (75.5, 78.0), turned to 90 degrees
- moved C45 4.00 mm to (185.0, 18.0)
- moved C46 4.00 mm to (180.0, 18.0)
- moved R69 4.00 mm to (190.0, 18.0)
- moved R70 4.00 mm to (195.0, 18.0)
- moved C49 3.61 mm to (198.0, 34.0)
- moved R71 3.61 mm to (198.0, 30.0)
- moved R72 3.61 mm to (177.0, 44.0)
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Routing:
- net V3V3: track 58.1 -> 2178.2 mm, vias 0 -> 85
- net ACTUATOR_12V: track 0.00 -> 705.7 mm, vias 0 -> 11
- net BANK_P_RAW: track 5.06 -> 603.7 mm, vias 0 -> 13
- net BUS_FUSED: track 4.68 -> 564.9 mm, vias 0 -> 11
- net RAIL_OK: track 0.00 -> 476.1 mm, vias 0 -> 8
- net REFEREE_PERMIT: track 0.00 -> 470.0 mm, vias 0 -> 17
- net V12_DRIVER: track 0.00 -> 457.0 mm, vias 0 -> 11
- net BYP_CAP_FB: track 0.00 -> 372.4 mm, vias 0 -> 11
- net CAP_ISO_COIL_M: track 0.00 -> 334.0 mm, vias 0 -> 7
- net PWM_AL: track 8.93 -> 310.1 mm, vias 0 -> 15
- net CAN_H: track 0.00 -> 289.6 mm
- net CAN_L: track 5.31 -> 293.3 mm
- net GATE_PERMIT: track 0.00 -> 286.1 mm, vias 0 -> 9
- net PRE_BUS_LED_P: track 0.00 -> 259.2 mm, vias 0 -> 2
- net PRE_BUS_LED_M: track 0.00 -> 258.2 mm, vias 0 -> 6
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