File: hardware/revb/control_board/charger.kicad_sch (KiCad schematic)
At the start: 51 parts, among them J1 XT30 input (PM chassis out), J2 XT30 chassis, J3 XT30 capacitor (to CM01), Q1 2N7002, Q2 2N7002 (inhibit), Q3 BSC059N04LS6 (Q1 HS buck), Q4 BSC059N04LS6 (Q2 LS buck), Q5 BSC059N04LS6 (Q3 HS boost), Q6 BSC059N04LS6 (Q4 LS boost), U1 LM5176PWPR

Commit message: hardware: tidy Rev B charger schematic layout (sections A-H), add PDF
Co-Authored-By: Claude Sonnet 5.5 <noreply@anthropic.com>
Claude-Session: https://claude.ai/code/session_0144JDnT2EZoCv7WaMs1JYhQ
Parts:
- C10: value 33n (Cc1) -> 10u/35V X7R; footprint Capacitor_SMD:C_0603_1608Metric -> Capacitor_SMD:C_1210_3225Metric
- C11: value 560p (Cc2) -> 10u/35V X7R; footprint Capacitor_SMD:C_0603_1608Metric -> Capacitor_SMD:C_1210_3225Metric
- C12: value 4.7u (VCC) -> 220p (SLOPE); footprint Capacitor_SMD:C_0805_2012Metric -> Capacitor_SMD:C_0603_1608Metric
- C13: value 0.22u (BOOT1) -> 0.1u (SS)
- C14: value 0.22u (BOOT2) -> 4.7u (VCC); footprint Capacitor_SMD:C_0603_1608Metric -> Capacitor_SMD:C_0805_2012Metric
- C15: value 10u/35V X7R -> 33n (Cc1); footprint Capacitor_SMD:C_1210_3225Metric -> Capacitor_SMD:C_0603_1608Metric
- C16: value 10u/35V X7R -> 560p (Cc2); footprint Capacitor_SMD:C_1210_3225Metric -> Capacitor_SMD:C_0603_1608Metric
- C17: value 10u/35V X7R -> 0.22u (BOOT1); footprint Capacitor_SMD:C_1210_3225Metric -> Capacitor_SMD:C_0603_1608Metric
- C18: value 10u/35V X7R -> 0.22u (BOOT2); footprint Capacitor_SMD:C_1210_3225Metric -> Capacitor_SMD:C_0603_1608Metric
- C8: value 220p (SLOPE) -> 10u/35V X7R; footprint Capacitor_SMD:C_0603_1608Metric -> Capacitor_SMD:C_1210_3225Metric
- C9: value 0.1u (SS) -> 10u/35V X7R; footprint Capacitor_SMD:C_0603_1608Metric -> Capacitor_SMD:C_1210_3225Metric
- Q4, Q5, Q6: footprint (none) -> Package_TO_SOT_SMD:Infineon_PG-TDSON-8_5.15x5.9mm
Connections:
- net BOOT1: now also C17.1; no longer C13.1
- net BOOT2: now also C18.1; no longer C14.1
- net COMP: now also C16.1; no longer C11.1
- net COMP_RC: now also C15.1; no longer C10.1
- net GND: now also C13.2, C14.2; no longer C17.2, C18.2
- net NODE: now also C10.1, C11.1, C8.1, C9.1; no longer C15.1, C16.1, C17.1, C18.1
- net SLOPE: now also C12.1; no longer C8.1
- net SS: now also C13.1; no longer C9.1
- net SW1: now also C17.2; no longer C13.2
- net SW2: now also C18.2; no longer C14.2
- net VCC_LM: now also C14.1; no longer C12.1
Other:
- note added: "A. Input / protection"
- note added: "B. Series PMOS (R2/R3 back-feed block)"
- note added: "C. Input current sense / input capacitors"
- note added: "Chassis and bank share this node. Bank via CM01."
- note added: "D. Output node (chassis + capacitor bank)"
- note added: "Default OFF. ON only when PMOS_EN=1 (Zener limits Vgs to 12V)."
- note added: "E. LM5176 settings"
- note added: "F. LM5176 controller"
- note added: "G. Gate drive"
- note added: "Gate resistors and bootstrap capacitors."
- note added: "H. Power stage"
- note added: "HTSSOP-28. Buck side = SW1/HDRV1/LDRV1, boost side = SW2/HDRV2/LDRV2."
- note added: "ISNS average limit 50mV/12mR = 4.2A (input power cap). Kelvin to ISNS+/-."
- note added: "PM chassis output 22-26V. Fuse + TVS (SMDJ30A)."
- note added: "Q1,Q2 = buck leg; Q3,Q4 = boost leg; one Rcs for both low sides (CS/CSG Kelvin)."
- note added: "Rev B control board: block 1 / charger (input protection, series PMOS, LM5176 4-switch buck-boost) - plan Y, PROVISIONAL"
- note added: "UVLO ~19V, no hiccup, 248kHz, Vout 26.2V."
- note added: "Values: docs/revb/plan_y_charger_sizing.md. Connectivity by net labels. Verify against the original datasheet: ISNS+/- polarity, MODE (hiccup), BIAS=NODE, UVLO values, FET/inductor footprints."
- note removed: "Rev B control board: block 1 (input protection, series PMOS, LM5176 4-switch buck-boost) PROVISIONAL (plan Y). Values: docs/revb/plan_y_charger_sizing.md. Connectivity by net labels. ISNS+/- polarity, MODE (hiccup), BIAS=NODE, UVLO values, FET footprints: verify against the original datasheet."

Commit message: Rev B: proper schematic symbols, block 2 (aux power, STM32G431, sensing, protection, CAN/UART), hierarchical root
Co-Authored-By: Claude Sonnet 5.5 <noreply@anthropic.com>
Claude-Session: https://claude.ai/code/session_0144JDnT2EZoCv7WaMs1JYhQ
Parts:
- removed C7: 100u/35V polymer, Capacitor_SMD:CP_Elec_8x10, symbol rev:C
- removed D1: TVS SMDJ30A, Diode_SMD:D_SMC, symbol rev:D
- removed D2: Zener 12V, Diode_SMD:D_SOD-123, symbol rev:D
- added C7: 100u/35V polymer, Capacitor_SMD:CP_Elec_8x10, symbol rev:CP
- added D1: TVS SMDJ30A (unidirectional), Diode_SMD:D_SMC, symbol rev:DZ
- added D2: Zener 12V (Vgs clamp), Diode_SMD:D_SOD-123, symbol rev:DZ
- added R18: 10mR 2512 (Rcs), Resistor_SMD:R_2512_6332Metric, symbol rev:R
- R10: value 10k (Rc1) -> 33k (RT, ~248kHz)
- R11: value 634k (RFB2, 26.2V) -> 10k (Rc1)
- R12: value 20k (RFB1) -> 634k (RFB2, 26.2V)
- R13: value 2R2 -> 20k (RFB1)
- R17: value 10mR 2512 (Rcs) -> 2R2; footprint Resistor_SMD:R_2512_6332Metric -> Resistor_SMD:R_0603_1608Metric; LCSC C2930473 -> (none); Note Kelvin to CS and CSG -> (none)
- R5: value 249k (RUV2) -> 2mR 2512 (cap-port shunt); footprint Resistor_SMD:R_0603_1608Metric -> Resistor_SMD:R_2512_6332Metric; Note (none) -> Kelvin to INA240 (control sheet)
- R6: value 17.4k (RUV1) -> 249k (RUV2); Note UVLO about 19V (provisional) -> (none)
- R7: value 100k (default inhibit) -> 17.4k (RUV1); Note (none) -> UVLO about 19V (provisional)
- R8: value 200k (MODE, no hiccup) -> 100k (default inhibit); Note 93.1k = hiccup enabled; undecided -> (none)
- R9: value 33k (RT, ~248kHz) -> 200k (MODE, no hiccup); Note (none) -> 93.1k = hiccup enabled; undecided
Connections:
- net CHG_INH: now also R8.1; no longer R7.1
- net COMP: now also R11.1; no longer R10.1
- net COMP_RC: now also R11.2; no longer R10.2
- net CS_N: now also R18.1; no longer R17.1
- net EN: now also R6.2, R7.1; no longer R5.2, R6.1
- net FB: now also R12.2, R13.1; no longer R11.2, R12.1
- net GND: now also R10.2, R13.2, R7.2, C7.2, D1.2 (A), R18.2; no longer R12.2, R17.2, R6.2, R8.2
- net HG1: now also R14.2; no longer R13.2
- net HG1_R: now also R14.1; no longer R13.1
- net HG2: now also R16.2; no longer R15.2
- net HG2_R: now also R16.1; no longer R15.1
- net LG1: now also R15.2; no longer R14.2
- net LG1_R: now also R15.1; no longer R14.1
- net LG2: now also R17.2; no longer R16.2
- net LG2_R: now also R17.1; no longer R16.1
- net MODE: now also R9.1; no longer R8.1
- net NODE: now also R12.1, R5.1; no longer J3.1 (+), R11.1
- net PG_GATE: now also D2.2 (A)
- net RT: now also R10.1; no longer R9.1
- net VCC_LM: no longer R7.2
- net VIN_C: now also R6.1, D2.1 (K); no longer R5.1
- net VIN_F: now also D1.1 (K)
- net VIN_P: now also C7.1
- new net 3V3: R8.2
- new net NODE_CAP: J3.1 (Pin_1), R5.2
