File: hardware/revb/control_board/buckboost.kicad_sch (KiCad schematic)
At the start: 41 parts, among them J101 XT30 chassis, J102 XT30 to CM01/bank, Q101 2N7002, Q102 60V N-MOS 5x6, Q103 60V N-MOS 5x6, Q104 60V N-MOS 5x6, Q105 60V N-MOS 5x6, U101 LM5176PWPR, U102 INA240A1PW

Commit message: Rev B control board: JLCPCB parts, 0402 passives, XT30 polarity fix, 4-layer PCB layout and routing
- parts chosen from JLCPCB stock (Basic/Preferred first), jlcpcb_bom.csv
- CAN connector 2-pin GH, XT30 pin1 = GND per AMASS footprint
- 68x57 mm 4-layer board, power pours + Freerouting + helper router
- KiCad 9 DRC: 0 errors, 0 unrouted; gerbers and CPL in fab/

Co-Authored-By: Claude Opus 5.5 <noreply@anthropic.com>
Claude-Session: https://claude.ai/code/session_0144JDnT2EZoCv7WaMs1JYhQ
Parts:
- C101: footprint Capacitor_SMD:C_0603_1608Metric -> Capacitor_SMD:C_0402_1005Metric; LCSC (none) -> C1530
- C102, C114: footprint Capacitor_SMD:C_0603_1608Metric -> Capacitor_SMD:C_0402_1005Metric; LCSC (none) -> C1525
- C103: value 560p -> 470p; footprint Capacitor_SMD:C_0603_1608Metric -> Capacitor_SMD:C_0402_1005Metric; LCSC (none) -> C1537
- C104: LCSC (none) -> C21117
- C105: value 4.7u 16V -> 4.7u 25V; LCSC (none) -> C1779
- C106, C107: LCSC (none) -> C14663
- C108, C109, C110, C111, C112: footprint Capacitor_SMD:C_1210_3225Metric -> Capacitor_SMD:C_1206_3216Metric; LCSC (none) -> C29823
- C113: footprint Capacitor_SMD:CP_Elec_10x10.5 -> Capacitor_SMD:CP_Elec_6.3x7.7; LCSC (none) -> C3151829; Note 50V hybrid polymer, part TBD -> 100u 50V Al electrolytic
- C115: footprint Capacitor_SMD:C_0603_1608Metric -> Capacitor_SMD:C_0402_1005Metric; LCSC (none) -> C1523
- D101: value SMDJ30A -> SMBJ30A; footprint Diode_SMD:D_SMC -> Diode_SMD:D_SMB; LCSC (none) -> C19077584
- J101, J102: footprint Connector_AMASS:AMASS_XT30PW-M_1x02_P2.50mm_Horizontal -> Connector_AMASS:AMASS_XT30UPB-M_1x02_P5.0mm_Vertical; LCSC (none) -> C428721
- L101: footprint Inductor_SMD:L_12x12mm_H8mm -> Inductor_SMD:L_Wuerth_HCI-1365; LCSC C6916222 -> C242228; Note MDA1360-100M, Isat >= 12 A, footprint to confirm -> SLO1365S100MTT 10uH Isat 12A 18mR; land pattern: verify vs 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
- Q101: LCSC (none) -> C8545
- Q102: value 60V N-MOS 5x6 -> NTMFS5C670NL; LCSC (none) -> C179626; Note 60V, Qg<=25nC, e.g. BSC028N06LS3 / TBD -> 60V 6.9mR 20nC SO-8FL
- Q103, Q104, Q105: value 60V N-MOS 5x6 -> NTMFS5C670NL; LCSC (none) -> C179626
- R101: value 249k -> 220k; footprint Resistor_SMD:R_0603_1608Metric -> Resistor_SMD:R_0402_1005Metric; LCSC (none) -> C25767
- R102: value 17.4k -> 15k; footprint Resistor_SMD:R_0603_1608Metric -> Resistor_SMD:R_0402_1005Metric; LCSC (none) -> C25756
- R103: footprint Resistor_SMD:R_0603_1608Metric -> Resistor_SMD:R_0402_1005Metric; LCSC (none) -> C25741
- R104: footprint Resistor_SMD:R_0603_1608Metric -> Resistor_SMD:R_0402_1005Metric; LCSC (none) -> C25764
- R105: footprint Resistor_SMD:R_0603_1608Metric -> Resistor_SMD:R_0402_1005Metric; LCSC (none) -> C25779
- R106: footprint Resistor_SMD:R_0603_1608Metric -> Resistor_SMD:R_0402_1005Metric; LCSC (none) -> C25744
- R107: value 634k 0.1% -> 1.5M; LCSC (none) -> C4172
- R108: value 20k 0.1% -> 47k; footprint Resistor_SMD:R_0603_1608Metric -> Resistor_SMD:R_0402_1005Metric; LCSC (none) -> C25792
- R109, R110, R111, R112: LCSC (none) -> C22939
- R113: value 10m 2512 -> 12m 2512; LCSC C2930473 -> C49164692
- R114: LCSC (none) -> C7420017
- R115: footprint Resistor_SMD:R_0603_1608Metric -> Resistor_SMD:R_0402_1005Metric; LCSC (none) -> C11702
- U102: LCSC (none) -> C93965
Connections:
- net GND: now also J101.1 (Pin_1), J102.1 (Pin_1); no longer J101.2 (Pin_2), J102.2 (Pin_2)
- net NODE: now also J101.2 (Pin_2); no longer J101.1 (Pin_1)
- net at R114.2, U102.3 (-): now also J102.2 (Pin_2); no longer J102.1 (Pin_1)
Other:
- note added: "C: 4.7u 50V X7R 1206 at the boost leg. D: clamps regen spikes if the bank is cut off."
- note added: "NODE = chassis output and capacitor bank (via CM01). fsw ~248 kHz (RT 33k), Vout 26.3 V (1.5M/47k), UVLO ~19.3 V (220k/15k), CCM, hiccup off (MODE 200k: confirm in datasheet)."
- note added: "Power FETs: 60 V class (input TVS SMBJ30A clamps up to ~48 V). Gate nets HG1/LG1/HG2/LG2 and SW1/SW2 are local labels; keep gate loops short in layout."
- note added: "Valley/peak current limits: buck 80 mV, boost 120 mV typ over 12 mR -> ~6.7 A / ~10 A inductor current (L Isat 12 A). CSLOPE 220p: recheck for Rcs 12 mR."
- note added: "Vout = 0.8 V x (1 + 1.5M/47k) = 26.33 V"
- note removed: "C: 4.7u 50V X7R 1210 at the boost leg. D: clamps regen spikes if the bank is cut off."
- note removed: "NODE = chassis output and capacitor bank (via CM01). fsw ~248 kHz (RT 33k), Vout 26.2 V (634k/20k), UVLO ~19 V, CCM, hiccup off (MODE 200k: confirm in datasheet)."
- note removed: "Power FETs: 60 V class (input TVS clamps up to ~48 V). Gate nets HG1/LG1/HG2/LG2 and SW1/SW2 are local labels; keep gate loops short in layout."
- note removed: "Valley/peak current limits: buck 80 mV, boost 120 mV typ over 10 mR -> ~8 A / ~12 A inductor current."
- note removed: "Vout = 0.8 V x (1 + 634k/20k) = 26.2 V"
