File: hardware/revb/control_board/mcu.kicad_sch (KiCad schematic)
At the start: 35 parts, among them J201 SWD 1.27mm, J202 CAN (GH 1.25 4p), J203 Referee (GH 1.25 3p), U201 AP63203WU, U202 STM32G431CBT6, U203 SN65HVD230, Y201 8MHz

Commit message: Rev B control board: JLCPCB parts, 0402 passives, XT30 polarity fix, 4-layer PCB layout and routing
- parts chosen from JLCPCB stock (Basic/Preferred first), jlcpcb_bom.csv
- CAN connector 2-pin GH, XT30 pin1 = GND per AMASS footprint
- 68x57 mm 4-layer board, power pours + Freerouting + helper router
- KiCad 9 DRC: 0 errors, 0 unrouted; gerbers and CPL in fab/

Co-Authored-By: Claude Opus 5.5 <noreply@anthropic.com>
Claude-Session: https://claude.ai/code/session_0144JDnT2EZoCv7WaMs1JYhQ
Parts:
- removed J202: CAN (GH 1.25 4p), Connector_JST:JST_GH_SM04B-GHS-TB_1x04-1MP_P1.25mm_Horizontal, symbol rev:CON4
- added J202: CAN (GH 1.25 2p), Connector_JST:JST_GH_SM02B-GHS-TB_1x02-1MP_P1.25mm_Horizontal, symbol rev:CON2
- C201, C202: footprint Capacitor_SMD:C_1210_3225Metric -> Capacitor_SMD:C_1206_3216Metric; LCSC (none) -> C13585
- C203, C206, C207, C208, C210, C214, C215: footprint Capacitor_SMD:C_0603_1608Metric -> Capacitor_SMD:C_0402_1005Metric; LCSC (none) -> C1525
- C204, C205: value 22u 10V -> 22u 25V; LCSC (none) -> C45783
- C209: footprint Capacitor_SMD:C_0603_1608Metric -> Capacitor_SMD:C_0402_1005Metric; LCSC (none) -> C52923
- C211: value 4.7u -> 4.7u 25V; LCSC (none) -> C1779
- C212, C213: value 12p -> 33p; footprint Capacitor_SMD:C_0603_1608Metric -> Capacitor_SMD:C_0402_1005Metric; LCSC (none) -> C1562
- D201, D202: LCSC (none) -> C8678
- D203: LCSC (none) -> C19077545
- D204: LCSC (none) -> C12624
- D205: LCSC (none) -> C2286
- J201: value SWD 1.27mm -> SWD 1.27mm (DNP); now not fitted
- J203: LCSC (none) -> C225126
- L201: footprint Inductor_SMD:L_Bourns-SRN4018 -> Inductor_SMD:L_Wuerth_MAPI-4030; LCSC (none) -> C167876; Note >=1A, part TBD -> FNR4030S6R8MT 4x4: verify land
- R201: footprint Resistor_SMD:R_0603_1608Metric -> Resistor_SMD:R_0402_1005Metric; LCSC (none) -> C25077
- R202: footprint Resistor_SMD:R_0603_1608Metric -> Resistor_SMD:R_0402_1005Metric; LCSC (none) -> C25744
- R203: footprint Resistor_SMD:R_0603_1608Metric -> Resistor_SMD:R_0402_1005Metric; LCSC (none) -> C25079; now not fitted
- R204, R205: footprint Resistor_SMD:R_0603_1608Metric -> Resistor_SMD:R_0402_1005Metric; LCSC (none) -> C25076
- R206, R207: footprint Resistor_SMD:R_0603_1608Metric -> Resistor_SMD:R_0402_1005Metric; LCSC (none) -> C11702
- U201: LCSC (none) -> C780769
- U203: LCSC (none) -> C12084
- Y201: footprint Crystal:Crystal_SMD_3225-4Pin_3.2x2.5mm -> Crystal:Crystal_SMD_5032-2Pin_5.0x3.2mm; LCSC (none) -> C115962; Note CL ~10pF, part TBD -> X50328MSB2GI CL 20pF
Connections:
- net at R203.2, U203.6 (CANL): now also J202.2 (Pin_2)
- net at R203.1, U203.7 (CANH): now also J202.1 (Pin_1)
- no-connect marks 17 -> 16
Other:
- note added: "Referee UART (3.3 V TTL)"
- note removed: "Referee UART (3.3 V TTL: confirm)"
