File: hardware/revb/control_board/power_input.kicad_sch (KiCad schematic)
At the start: 27 parts, among them J1 XT30, Q1 AOD409, Q2 2N7002, Q3 MMBT5551, U1 INA240A1PW

Commit message: Rev B control board: JLCPCB parts, 0402 passives, XT30 polarity fix, 4-layer PCB layout and routing
- parts chosen from JLCPCB stock (Basic/Preferred first), jlcpcb_bom.csv
- CAN connector 2-pin GH, XT30 pin1 = GND per AMASS footprint
- 68x57 mm 4-layer board, power pours + Freerouting + helper router
- KiCad 9 DRC: 0 errors, 0 unrouted; gerbers and CPL in fab/

Co-Authored-By: Claude Opus 5.5 <noreply@anthropic.com>
Claude-Session: https://claude.ai/code/session_0144JDnT2EZoCv7WaMs1JYhQ
Parts:
- C1, C2, C3, C4, C5, C6: footprint Capacitor_SMD:C_1210_3225Metric -> Capacitor_SMD:C_1206_3216Metric; LCSC (none) -> C29823
- C10: footprint Capacitor_SMD:C_0603_1608Metric -> Capacitor_SMD:C_0402_1005Metric; LCSC (none) -> C1523
- C7: footprint Capacitor_SMD:CP_Elec_10x10.5 -> Capacitor_SMD:CP_Elec_6.3x7.7; LCSC (none) -> C3151829; Note hybrid polymer, part TBD -> (none)
- C8, C9: footprint Capacitor_SMD:C_0603_1608Metric -> Capacitor_SMD:C_0402_1005Metric; LCSC (none) -> C1525
- D1: value SMDJ30A -> SMBJ30A; footprint Diode_SMD:D_SMC -> Diode_SMD:D_SMB; LCSC (none) -> C19077584
- D2: LCSC (none) -> C19077426
- F1: footprint Fuse:Fuse_2920_7451Metric -> Fuse:Fuse_1206_3216Metric; LCSC (none) -> C52988557; Note part TBD (fast, >=10A, 32V) -> LTC1206-2100TS 10A 32V
- J1: footprint Connector_AMASS:AMASS_XT30PW-M_1x02_P2.50mm_Horizontal -> Connector_AMASS:AMASS_XT30UPB-M_1x02_P5.0mm_Vertical; LCSC (none) -> C428721; Note from PM chassis output -> from PM chassis output. pin1 = -, pin2 = + (AMASS)
- Q2: LCSC (none) -> C8545
- Q3: LCSC (none) -> C2145
- R1, R3, R8: footprint Resistor_SMD:R_0603_1608Metric -> Resistor_SMD:R_0402_1005Metric; LCSC (none) -> C25741
- R2: footprint Resistor_SMD:R_0603_1608Metric -> Resistor_SMD:R_0402_1005Metric; LCSC (none) -> C25744
- R4: LCSC (none) -> C49164692
- R5: footprint Resistor_SMD:R_0603_1608Metric -> Resistor_SMD:R_0402_1005Metric; LCSC (none) -> C25076
- R6: footprint Resistor_SMD:R_0603_1608Metric -> Resistor_SMD:R_0402_1005Metric; LCSC (none) -> C25917
- R7, R9: footprint Resistor_SMD:R_0603_1608Metric -> Resistor_SMD:R_0402_1005Metric; LCSC (none) -> C11702
- U1: LCSC (none) -> C93965
Connections:
- net GND: now also J1.1 (Pin_1); no longer J1.2 (Pin_2)
- net at F1.1: now also J1.2 (Pin_2); no longer J1.1 (Pin_1)
Other:
- note added: "C1-C6: 4.7u 50V X7R 1206. C7: 100u 50V Al electrolytic. Place at the buck leg (Q101/Q102)."
- note removed: "C1-C6: 4.7u 50V X7R 1210. C7: 100u 50V hybrid polymer. Place at the buck leg (Q101/Q102)."
