File: hardware/revb/control_board/protect_sense.kicad_sch (KiCad schematic)
At the start: 34 parts, among them Q301 2N7002, Q302 2N7002, Q303 2N7002, U301 TL431 (2.495 V), U302 LM393

Commit message: Rev B control board: JLCPCB parts, 0402 passives, XT30 polarity fix, 4-layer PCB layout and routing
- parts chosen from JLCPCB stock (Basic/Preferred first), jlcpcb_bom.csv
- CAN connector 2-pin GH, XT30 pin1 = GND per AMASS footprint
- 68x57 mm 4-layer board, power pours + Freerouting + helper router
- KiCad 9 DRC: 0 errors, 0 unrouted; gerbers and CPL in fab/

Co-Authored-By: Claude Opus 5.5 <noreply@anthropic.com>
Claude-Session: https://claude.ai/code/session_0144JDnT2EZoCv7WaMs1JYhQ
Parts:
- C301, C302, C303, C304, C307: footprint Capacitor_SMD:C_0603_1608Metric -> Capacitor_SMD:C_0402_1005Metric; LCSC (none) -> C1525
- C305, C306: footprint Capacitor_SMD:C_0603_1608Metric -> Capacitor_SMD:C_0402_1005Metric; LCSC (none) -> C1523
- Q301, Q302, Q303: LCSC (none) -> C8545
- R301, R303, R313, R319, R321: footprint Resistor_SMD:R_0603_1608Metric -> Resistor_SMD:R_0402_1005Metric; LCSC (none) -> C25741
- R302, R304, R305, R307, R308, R311, R315, R317: footprint Resistor_SMD:R_0603_1608Metric -> Resistor_SMD:R_0402_1005Metric; LCSC (none) -> C25744
- R306: LCSC (none) -> C23204
- R309: value 100k -> 150k; footprint Resistor_SMD:R_0603_1608Metric -> Resistor_SMD:R_0402_1005Metric; LCSC (none) -> C25755
- R310: value 4.53k 1% -> 6.8k; footprint Resistor_SMD:R_0603_1608Metric -> Resistor_SMD:R_0402_1005Metric; LCSC (none) -> C25917
- R312, R316: footprint Resistor_SMD:R_0603_1608Metric -> Resistor_SMD:R_0402_1005Metric; LCSC (none) -> C26083
- R314: value 4.75k 1% -> 4.7k; footprint Resistor_SMD:R_0603_1608Metric -> Resistor_SMD:R_0402_1005Metric; LCSC (none) -> C25900
- R318: footprint Resistor_SMD:R_0603_1608Metric -> Resistor_SMD:R_0402_1005Metric; LCSC (none) -> C25900
- R320: footprint Resistor_SMD:R_0603_1608Metric -> Resistor_SMD:R_0402_1005Metric; LCSC (none) -> C11702
- TH301: value NTC 10k B3950 -> NTC 10k B3380; LCSC (none) -> C13564
- U301: LCSC (none) -> C181103
- U302: LCSC (none) -> C7955
Other:
- note added: "Node OV 27.8 V -> NODE_OK low (converter off)"
- note removed: "Node OV 27.5 V -> NODE_OK low (converter off)"
